Commit message: Running Version : 5/12/16

File: urdf/decorations.urdf.xacro (robot description, xacro)
@@ -21,6 +21,6 @@
 ARISING IN ANY WAY OUT OF THE USE OF THIS SOFTWARE, EVEN IF ADVISED OF THE POSSIBILITY OF SUCH DAMAGE.
 -->
-<robot name="mars_rover_decorations" xmlns:xacro="http://ros.org/wiki/xacro">
-  <xacro:macro name="rover_decorate">
+<robot name="husky_decorations" xmlns:xacro="http://ros.org/wiki/xacro">
+  <xacro:macro name="husky_decorate">
     <!-- Spawn Husky chassis -->
     <link name="top_chassis_link">
@@ -28,5 +28,5 @@
         <origin xyz="0 0 0" rpy="0 0 0" />
         <geometry>
-          <mesh filename="package://msi_2k16_17_urdf/meshes/top_chassis.dae" />
+          <mesh filename="package://husky_description/meshes/top_chassis.dae" />
         </geometry>
       </visual>
@@ -41,5 +41,5 @@
       <visual>
         <geometry>
-          <mesh filename="package://msi_2k16_17_urdf/meshes/user_rail.dae" />
+          <mesh filename="package://husky_description/meshes/user_rail.dae" />
         </geometry>
       </visual>
@@ -55,5 +55,5 @@
       <visual>
         <geometry>
-          <mesh filename="package://msi_2k16_17_urdf/meshes/bumper.dae" />
+          <mesh filename="package://husky_description/meshes/bumper.dae" />
         </geometry>
       </visual>
@@ -69,5 +69,5 @@
       <visual>
         <geometry>
-          <mesh filename="package://msi_2k16_17_urdf/meshes/bumper.dae" />
+          <mesh filename="package://husky_description/meshes/bumper.dae" />
         </geometry>
       </visual>
@@ -84,5 +84,5 @@
           <origin xyz="0 0 0" rpy="0 0 0" />
           <geometry>
-            <mesh filename="package://msi_2k16_17_urdf/meshes/top_plate.dae" />
+            <mesh filename="package://husky_description/meshes/top_plate.dae" />
           </geometry>
         </visual>
@@ -90,5 +90,5 @@
           <origin xyz="0 0 0" rpy="0 0 0"/>
           <geometry>
-            <mesh filename="package://msi_2k16_17_urdf/meshes/top_plate.dae" />
+            <mesh filename="package://husky_description/meshes/top_plate.dae" />
           </geometry>
         </collision>

File: urdf/msi.xacro (robot description, xacro)
@@ -4,5 +4,5 @@
   <xacro:include filename="$(find husky_description)/urdf/decorations.urdf.xacro" />
   <xacro:include filename="$(find husky_description)/urdf/wheel.urdf.xacro" />
-  <xacro:include filename="$(find ur_description)/urdf/ur5.urdf.xacro" />
+  <!--<xacro:include filename="$(find ur_description)/urdf/ur5.urdf.xacro" />-->
   <property name="M_PI" value="3.14159"/>
   <!-- Base Size -->
@@ -103,10 +103,11 @@
       <xacro:property name="reflect" value="-1" />
       <!-- Spawn arm -->
-      <xacro:ur5_robot prefix="ur5_arm_" joint_limited="true"/>
+<!--    <xacro:ur5_robot prefix="ur5_arm_" joint_limited="true"/> -->
       <!-- Join arm -->
-      <joint name="ur5_arm_base" type="fixed">
+<!--      <joint name="ur5_arm_base" type="fixed">
         <parent link="top_plate_link" />
         <child link="ur5_arm_base_link" />
         <origin xyz="0.3058 0 0.0065" rpy="0.0 0.0 -1.57" />
       </joint>
+-->
 </robot>

File: urdf/wheel.urdf.xacro (robot description, xacro)
@@ -21,21 +21,20 @@
 ARISING IN ANY WAY OUT OF THE USE OF THIS SOFTWARE, EVEN IF ADVISED OF THE POSSIBILITY OF SUCH DAMAGE.
 -->
-<robot xmlns:xacro="http://ros.org/wiki/xacro" name="rover_wheel">
-	<xacro:macro name="rover_wheel" params="wheel_prefix *joint_pose">
+<robot xmlns:xacro="http://ros.org/wiki/xacro" name="husky_wheel">
+	<xacro:macro name="husky_wheel" params="wheel_prefix *joint_pose">
 		<link name="${wheel_prefix}_wheel_link">
 			<inertial>
 				<mass value="2.637" />
-				<origin xyz="0 0 0" />
+				<xacro:insert_block name="joint_pose"/>
 				<inertia  ixx="0.02467" ixy="0" ixz="0" iyy="0.02467" iyz="0" izz="0.04411" />
 			</inertial>
 			<visual>
-				<origin xyz="0 0 0" rpy="0 0 0" />
+				<xacro:insert_block name="joint_pose"/>
 				<geometry>
-					<!--<mesh filename="package://msi_2k16_17_urdf/meshes/wheel.dae" />-->
-					        <cylinder radius="0.2" length="0.6"/>
+					<mesh filename="package://husky_description/meshes/wheel.dae" />
 				</geometry>
 			</visual>
 			<collision>
-				<origin xyz="0 0 0" rpy="${M_PI/2} 0 0" />
+				<xacro:insert_block name="joint_pose"/>
 				<geometry>
 					<cylinder length="${wheel_length}" radius="${wheel_radius}" />
