Commit message: Husky is a sucks

File: msi_2k16_17_urdf/urdf/decorations.urdf.xacro (robot description, xacro)
@@ -28,5 +28,5 @@
         <origin xyz="0 0 0" rpy="0 0 0" />
         <geometry>
-          <mesh filename="package://husky_description/meshes/top_chassis.dae" />
+          <mesh filename="package://msi_2k16_17_urdf/meshes/top_chassis.dae" />
         </geometry>
       </visual>
@@ -41,5 +41,5 @@
       <visual>
         <geometry>
-          <mesh filename="package://husky_description/meshes/user_rail.dae" />
+          <mesh filename="package://msi_2k16_17_urdf/meshes/user_rail.dae" />
         </geometry>
       </visual>
@@ -55,5 +55,5 @@
       <visual>
         <geometry>
-          <mesh filename="package://husky_description/meshes/bumper.dae" />
+          <mesh filename="package://msi_2k16_17_urdf/meshes/bumper.dae" />
         </geometry>
       </visual>
@@ -69,5 +69,5 @@
       <visual>
         <geometry>
-          <mesh filename="package://husky_description/meshes/bumper.dae" />
+          <mesh filename="package://msi_2k16_17_urdf/meshes/bumper.dae" />
         </geometry>
       </visual>
@@ -84,5 +84,5 @@
           <origin xyz="0 0 0" rpy="0 0 0" />
           <geometry>
-            <mesh filename="package://husky_description/meshes/top_plate.dae" />
+            <mesh filename="package://msi_2k16_17_urdf/meshes/top_plate.dae" />
           </geometry>
         </visual>
@@ -90,5 +90,5 @@
           <origin xyz="0 0 0" rpy="0 0 0"/>
           <geometry>
-            <mesh filename="package://husky_description/meshes/top_plate.dae" />
+            <mesh filename="package://msi_2k16_17_urdf/meshes/top_plate.dae" />
           </geometry>
         </collision>

File: msi_2k16_17_urdf/urdf/msi.xacro (robot description, xacro)
@@ -2,44 +2,31 @@
 <robot name="mars_rover_iitb" xmlns:xacro="http://ros.org/wiki/xacro">
   <!-- Included URDF/XACRO Files -->
-  <xacro:include filename="$(find husky_description)/urdf/decorations.urdf.xacro" />
-  <xacro:include filename="$(find husky_description)/urdf/wheel.urdf.xacro" />
+  <!-- <xacro:include filename="$(find msi_2k16_17_urdf)/urdf/decorations.urdf.xacro" /> -->
+  <xacro:include filename="$(find msi_2k16_17_urdf)/urdf/wheel.urdf.xacro" />
   <!--<xacro:include filename="$(find ur_description)/urdf/ur5.urdf.xacro" />-->
   <property name="M_PI" value="3.14159"/>
   <!-- Base Size -->
-  <property name="base_x_size" value="1.5" />
-  <property name="base_y_size" value="0.97090000" />
-  <property name="base_z_size" value="0.4750000" />
+  <property name="base_x_size" value="1.1" />
+  <property name="base_y_size" value="0.55" />
+  <property name="base_z_size" value="0.35" />
+  <!-- Wheel Properties -->
+  <property name="wheel_L" value="0.11" />
+  <property name="wheel_R" value="0.17" />
   <!-- Wheel Mounting Positions -->
-  <xacro:property name="wheelbase" value="1.3" />
-  <xacro:property name="track" value="0.9708" />
-  <xacro:property name="wheel_vertical_offset" value="0.03282" />
-  <!-- Wheel Properties -->
-  <xacro:property name="wheel_length" value="0.20" />
-  <xacro:property name="wheel_radius" value="0.225" />
+  <xacro:property name="wheelbase" value="0.54" />
+  <xacro:property name="track" value="0.375" />
+  <xacro:property name="wheel_vertical_offset" value="${-base_z_size/4}" />
     <!-- Base link is the center of the robot's bottom plate -->
-    <link name="base_link">
-      <visual>
-        <origin xyz="0 0 0" rpy="0 0 0" />
-        <geometry>
-          <mesh filename="package://husky_description/meshes/base_link.dae" />
-        </geometry>
-      </visual>
-      <collision>
-        <origin xyz="0 0 ${base_z_size/4}" rpy="0 0 0" />
-        <geometry>
-          <box size="${base_x_size} ${base_y_size} ${base_z_size/2}"/>
-        </geometry>
-      </collision>
-      <collision>
-        <origin xyz="0 0 ${base_z_size*3/4}" rpy="0 0 0" />
-        <geometry>
-          <box size="${base_x_size*4/5} ${base_y_size} ${base_z_size/2}"/>
-        </geometry>
-      </collision>
-    </link>
+  <link name="base_link">
+    <visual>
+      <geometry>
+        <box size="${base_x_size} ${base_y_size} ${base_z_size}"/>
+      </geometry>
+    </visual>
+  </link>
     <!-- Base footprint is on the ground under the robot -->
     <link name="base_footprint"/>
     <joint name="base_footprint_joint" type="fixed">
-      <origin xyz="0 0 ${wheel_vertical_offset - wheel_radius}" rpy="0 0 0" />
+      <origin xyz="0 0 ${wheel_vertical_offset}" rpy="0 0 0" />
       <parent link="base_link" />
       <child link="base_footprint" />
@@ -69,7 +56,4 @@
     </gazebo>
     <!-- wheel macros -->
-    <xacro:property name="front_left_origin">
- 	 <origin xyz="${wheelbase/2} ${track/2} ${wheel_vertical_offset}" rpy="0 0 0" />
-	</xacro:property>
 <xacro:property name="front_right_origin">
  	 <origin xyz="${wheelbase/2} ${-track/2} ${wheel_vertical_offset}" rpy="0 0 0" />
@@ -81,24 +65,24 @@
  	 <origin xyz="${-wheelbase/2} ${-track/2} ${wheel_vertical_offset}" rpy="0 0 0" />
 	</xacro:property>
-    <xacro:husky_wheel wheel_prefix="front_left">
+<xacro:husky_wheel wheel_prefix="front_left">
 	<origin xyz="${wheelbase/2} ${track/2} ${wheel_vertical_offset}" rpy="0 0 0" />
 	</xacro:husky_wheel>
-    <xacro:husky_wheel wheel_prefix="front_right">
-<origin xyz="${wheelbase/2} ${-track/2} ${wheel_vertical_offset}" rpy="0 0 0" />
+<xacro:husky_wheel wheel_prefix="front_right">
+	<origin xyz="${wheelbase/2} ${-track/2} ${wheel_vertical_offset}" rpy="0 0 0" />
 </xacro:husky_wheel>
-    <xacro:husky_wheel wheel_prefix="rear_left" >
- <origin xyz="${-wheelbase/2} ${track/2} ${wheel_vertical_offset}" rpy="0 0 0" />
+<xacro:husky_wheel wheel_prefix="rear_left" >
+	<origin xyz="${-wheelbase/2} ${track/2} ${wheel_vertical_offset}" rpy="0 0 0" />
 </xacro:husky_wheel>
-    <xacro:husky_wheel wheel_prefix="rear_right">
-<origin xyz="${-wheelbase/2} ${-track/2} ${wheel_vertical_offset}" rpy="0 0 0" />
+<xacro:husky_wheel wheel_prefix="rear_right">
+	<origin xyz="${-wheelbase/2} ${-track/2} ${wheel_vertical_offset}" rpy="0 0 0" />
 </xacro:husky_wheel>
-   <xacro:husky_wheel wheel_prefix="center_left" >
- <origin xyz="0 ${track/2} ${wheel_vertical_offset}" rpy="0 0 0" />
+<xacro:husky_wheel wheel_prefix="center_left" >
+	<origin xyz="0 ${track/2} ${wheel_vertical_offset}" rpy="0 0 0" />
 </xacro:husky_wheel>
-    <xacro:husky_wheel wheel_prefix="center_right">
-<origin xyz="0 ${-track/2} ${wheel_vertical_offset}" rpy="0 0 0" />
+<xacro:husky_wheel wheel_prefix="center_right">
+	<origin xyz="0 ${-track/2} ${wheel_vertical_offset}" rpy="0 0 0" />
 </xacro:husky_wheel>
     <!-- Decorations MAcro -->
-    <xacro:husky_decorate />
+<xacro:husky_decorate />
       <xacro:property name="reflect" value="-1" />
       <!-- Spawn arm -->

File: msi_2k16_17_urdf/urdf/wheel.urdf.xacro (robot description, xacro)
@@ -32,5 +32,5 @@
 				<xacro:insert_block name="joint_pose"/>
 				<geometry>
-					<mesh filename="package://husky_description/meshes/wheel.dae" />
+					<mesh filename="package://msi_2k16_17_urdf/meshes/wheel.dae" />
 				</geometry>
 			</visual>
@@ -38,5 +38,5 @@
 				<xacro:insert_block name="joint_pose"/>
 				<geometry>
-					<cylinder length="${wheel_length}" radius="${wheel_radius}" />
+					<cylinder length="${wheel_L}" radius="${wheel_R}" />
 				</geometry>
 			</collision>
