Commit message: Rocker-Bogie done

File: msi_2k16_17_urdf/urdf/arm.urdf (robot description, URDF)
Before this commit: robot jaco, 12 links, 11 joints
Joints:
- joint jaco_finger_joint_1: limit lower=0.004 upper=1.044 effort=30 velocity=5 -> lower=0.001 upper=0.5 effort=30 velocity=1
- joint jaco_finger_joint_2: limit lower=0.004 upper=1.044 effort=30 velocity=5 -> lower=0.004 upper=0.5 effort=30 velocity=1
- joint jaco_finger_joint_3: limit lower=0.004 upper=1.044 effort=30 velocity=5 -> lower=0.004 upper=0.5 effort=30 velocity=1
- joint jaco_joint_1: limit lower=-3.14159265359 upper=3.14159265359 effort=30 velocity=5 -> lower=-1.57 upper=1.57 effort=30 velocity=1
- joint jaco_joint_2: limit lower=-3.14159265359 upper=3.14159265359 effort=30 velocity=5 -> lower=-1.57 upper=1.57 effort=30 velocity=1
- joint jaco_joint_3: limit lower=-3.14159265359 upper=3.14159265359 effort=30 velocity=5 -> lower=-1.57 upper=1.57 effort=30 velocity=1
- joint jaco_joint_4: limit lower=-3.14159265359 upper=3.14159265359 effort=30 velocity=5 -> lower=-1.57 upper=1.57 effort=30 velocity=1
- joint jaco_joint_5: limit lower=-3.14159265359 upper=3.14159265359 effort=30 velocity=5 -> lower=-1.57 upper=1.57 effort=30 velocity=1
- joint jaco_joint_6: limit lower=-3.14159265359 upper=3.14159265359 effort=30 velocity=5 -> lower=-1.57 upper=1.57 effort=30 velocity=1

File: msi_2k16_17_urdf/urdf/msi.xacro (robot description, xacro)
@@ -11,5 +11,5 @@
   <!-- Base Size -->
   <property name="base_x_size" value="1.1" />
-  <property name="base_y_size" value="0.55" />
+  <property name="base_y_size" value="0.59" />
   <property name="base_z_size" value="0.35" />
   <!-- Wheel Properties -->
@@ -20,5 +20,5 @@
   <!-- Wheel Mounting Positions -->
   <xacro:property name="wheelbase" value="1.08" />
-  <xacro:property name="track" value="0.75" />
+  <xacro:property name="track" value="1.0" />
   <xacro:property name="wheel_vertical_offset" value="${-base_z_size/2}" />
     <!-- Base link is the center of the robot's bottom plate -->
@@ -32,4 +32,100 @@
     </visual>
   </link>
+  <link name="rocker_left">
+     <visual>
+      <geometry>
+         <mesh filename="package://msi_2k16_17_urdf/meshes/rocker.stl" scale="0.01 0.01 0.01"/>
+      </geometry>
+      <origin xyz="0 0 0" rpy="0 0 0"/>
+      <material name="chassis"/>
+    </visual>
+    <inertial>
+      <origin xyz="0 0 1" rpy="0 0 0"/>
+      <mass value="1"/>
+      <inertia
+        ixx="1.0" ixy="0.0" ixz="0.0"
+        iyy="1.0" iyz="0.0"
+        izz="1.0"/>
+    </inertial>
+  </link>
+  <joint name="rocker_left_to_chassis" type="revolute">
+      <origin xyz=" 0 ${base_y_size/2 + 0.07} 0" rpy="0 0 0"/>
+      <parent link="base_link"/>
+      <child link="rocker_left"/>
+<limit effort="100" lower="-0.17" upper="0.17" velocity="1"/>
+      <axis xyz="0 1 0" rpy="0 0 0" />
+  </joint>
+  <link name="rocker_right">
+     <visual>
+      <geometry>
+         <mesh filename="package://msi_2k16_17_urdf/meshes/rocker.stl" scale="0.01 0.01 0.01"/>
+      </geometry>
+      <origin xyz="0 0 0" rpy="0 0 0"/>
+      <material name="chassis"/>
+    </visual>
+    <inertial>
+      <origin xyz="0 0 1" rpy="0 0 0"/>
+      <mass value="1"/>
+      <inertia
+        ixx="1.0" ixy="0.0" ixz="0.0"
+        iyy="1.0" iyz="0.0"
+        izz="1.0"/>
+    </inertial>
+  </link>
+  <joint name="rocker_right_to_chassis" type="revolute">
+      <origin xyz=" 0 ${-base_y_size/2 - 0.02} 0" rpy="0 0 0"/>
+      <parent link="base_link"/>
+      <child link="rocker_right"/>
+<limit effort="100" lower="-0.17" upper="0.17" velocity="1"/>
+      <axis xyz="0 1 0" rpy="0 0 0" />
+  </joint>
+  <link name="bogie_left">
+    <visual>
+     <geometry>
+       <mesh filename="package://msi_2k16_17_urdf/meshes/bogie.stl" scale="0.01 0.01 0.01"/>
+     </geometry>
+      <origin xyz="-0.202 -0.0444 -0.1434" rpy="0 0 0"/>
+      <material name="chassis"/>
+    </visual>
+    <inertial>
+      <origin xyz="0 0 1" rpy="0 0 0"/>
+      <mass value="1"/>
+      <inertia
+        ixx="1.0" ixy="0.0" ixz="0.0"
+        iyy="1.0" iyz="0.0"
+        izz="1.0"/>
+    </inertial>
+  </link>
+  <joint name="bogie_left_to_rocker" type="revolute">
+      <origin xyz="0 0 0 " rpy="0 0 0"/>
+      <parent link="rocker_left"/>
+      <child link="bogie_left"/>
+<limit effort="100" lower="-0.17" upper="0.17" velocity="1"/>
+      <axis xyz="0 1 0" rpy="0 0 0" />
+  </joint>
+  <link name="bogie_right">
+    <visual>
+     <geometry>
+       <mesh filename="package://msi_2k16_17_urdf/meshes/bogie.stl" scale="0.01 0.01 0.01"/>
+     </geometry>
+      <origin xyz="-0.202 -0.044 -0.1434 " rpy="0 0 0"/>
+      <material name="chassis"/>
+    </visual>
+    <inertial>
+      <origin xyz="0 0 1" rpy="0 0 0"/>
+      <mass value="1"/>
+      <inertia
+        ixx="1.0" ixy="0.0" ixz="0.0"
+        iyy="1.0" iyz="0.0"
+        izz="1.0"/>
+    </inertial>
+  </link>
+  <joint name="bogie_right_to_roc" type="revolute">
+      <origin xyz="0 0 0" rpy="0 0 0"/>
+      <parent link="rocker_right"/>
+      <child link="bogie_right"/>
+<limit effort="100" lower="-0.17" upper="0.17" velocity="1"/>
+      <axis xyz="0 1 0" rpy="0 0 0" />
+  </joint>
     <!-- Base footprint is on the ground under the robot -->
     <link name="base_footprint"/>

Commit message: Done and Dusted

File: msi_2k16_17_urdf/urdf/arm.urdf (robot description, URDF)
Before this commit: robot jaco, 12 links, 11 joints
Joints:
- joint jaco_finger_joint_1: limit lower=0.001 upper=0.5 effort=30 velocity=1 -> lower=0.001 upper=0.5 effort=10 velocity=1
- joint jaco_finger_joint_2: limit lower=0.004 upper=0.5 effort=30 velocity=1 -> lower=0.004 upper=0.5 effort=10 velocity=1
- joint jaco_finger_joint_3: limit lower=0.004 upper=0.5 effort=30 velocity=1 -> lower=0.004 upper=0.5 effort=10 velocity=1
- joint jaco_joint_1: limit lower=-1.57 upper=1.57 effort=30 velocity=1 -> lower=-0.2 upper=0.2 effort=10 velocity=1
- joint jaco_joint_2: limit lower=-1.57 upper=1.57 effort=30 velocity=1 -> lower=-0.6 upper=0.65 effort=10 velocity=1
- joint jaco_joint_3: limit lower=-1.57 upper=1.57 effort=30 velocity=1 -> lower=-0.1 upper=0.1 effort=10 velocity=1
- joint jaco_joint_4: limit lower=-1.57 upper=1.57 effort=30 velocity=1 -> lower=2.44 upper=2.46 effort=10 velocity=1
- joint jaco_joint_5: limit lower=-1.57 upper=1.57 effort=30 velocity=1 -> lower=2.48 upper=2.5 effort=10 velocity=1
- joint jaco_joint_6: limit lower=-1.57 upper=1.57 effort=30 velocity=1 -> lower=1.86 upper=1.88 effort=10 velocity=1

File: msi_2k16_17_urdf/urdf/msi.xacro (robot description, xacro)
@@ -38,4 +38,7 @@
     </visual>
   </link>
+  <gazebo reference="base_link">
+    <material> Gazebo/Grey</material>
+  </gazebo>
   <link name="rocker_R">
      <visual>

File: msi_2k16_17_urdf/urdf/wheel.urdf.xacro (robot description, xacro)
@@ -48,4 +48,5 @@
 			<kd value="1.0" />
 			<fdir1 value="1 0 0"/>
+    		<material> Gazebo/FlatBlack</material>
 		</gazebo>
 		<joint name="${wheel_prefix}_wheel" type="continuous">
