Commit message: Implemented Parameter Passing across Macros

File: msi_2k16_17_urdf/urdf/msi.xacro (robot description, xacro)
@@ -2,23 +2,19 @@
 <robot name="mars_rover_iitb" xmlns:xacro="http://ros.org/wiki/xacro">
   <!-- Included URDF/XACRO Files -->
-  <xacro:include filename="$(find msi_2k16_17_urdf)/urdf/decorations.urdf.xacro" />
-  <create/>
-  <xacro:include filename="$(find msi_2k16_17_urdf)/urdf/wheel.urdf.xacro" />
-  <create/>
+  <xacro:include filename="$(find husky_description)/urdf/decorations.urdf.xacro" />
+  <xacro:include filename="$(find husky_description)/urdf/wheel.urdf.xacro" />
   <xacro:include filename="$(find ur_description)/urdf/ur5.urdf.xacro" />
-  <create/>
   <property name="M_PI" value="3.14159"/>
   <!-- Base Size -->
-  <property name="base_x_size" value="0.98740000" />
-  <property name="base_y_size" value="0.57090000" />
-  <property name="base_z_size" value="0.24750000" />
+  <property name="base_x_size" value="1.5" />
+  <property name="base_y_size" value="0.97090000" />
+  <property name="base_z_size" value="0.4750000" />
   <!-- Wheel Mounting Positions -->
-  <xacro:property name="wheelbase" value="0.5120" />
-  <xacro:property name="track" value="0.5708" />
+  <xacro:property name="wheelbase" value="1.3" />
+  <xacro:property name="track" value="0.9708" />
   <xacro:property name="wheel_vertical_offset" value="0.03282" />
   <!-- Wheel Properties -->
-  <xacro:property name="wheel_length" value="0.1143" />
-  <xacro:property name="wheel_radius" value="0.17775" />
-  <xacro:macro name="mars_rover_iitb">
+  <xacro:property name="wheel_length" value="0.20" />
+  <xacro:property name="wheel_radius" value="0.225" />
     <!-- Base link is the center of the robot's bottom plate -->
     <link name="base_link">
@@ -26,5 +22,5 @@
         <origin xyz="0 0 0" rpy="0 0 0" />
         <geometry>
-          <mesh filename="$(find msi_2k16_17_urdf)/meshes/base_link.dae" />
+          <mesh filename="package://husky_description/meshes/base_link.dae" />
         </geometry>
       </visual>
@@ -73,18 +69,36 @@
     </gazebo>
     <!-- wheel macros -->
-    <xacro:rover_wheel wheel_prefix="front_left">
-      <origin xyz="${wheelbase/2} ${track/2} ${wheel_vertical_offset}" rpy="0 0 0" />
-    </xacro:rover_wheel>
-    <xacro:rover_wheel wheel_prefix="front_right">
-      <origin xyz="${wheelbase/2} ${-track/2} ${wheel_vertical_offset}" rpy="0 0 0" />
-    </xacro:rover_wheel>
-    <xacro:rover_wheel wheel_prefix="rear_left">
-      <origin xyz="${-wheelbase/2} ${track/2} ${wheel_vertical_offset}" rpy="0 0 0" />
-    </xacro:rover_wheel>
-    <xacro:rover_wheel wheel_prefix="rear_right">
-      <origin xyz="${-wheelbase/2} ${-track/2} ${wheel_vertical_offset}" rpy="0 0 0" />
-    </xacro:rover_wheel>
+    <xacro:property name="front_left_origin">
+ 	 <origin xyz="${wheelbase/2} ${track/2} ${wheel_vertical_offset}" rpy="0 0 0" />
+	</xacro:property>
+<xacro:property name="front_right_origin">
+ 	 <origin xyz="${wheelbase/2} ${-track/2} ${wheel_vertical_offset}" rpy="0 0 0" />
+	</xacro:property>
+<xacro:property name="rear_left_origin">
+ 	 <origin xyz="${-wheelbase/2} ${track/2} ${wheel_vertical_offset}" rpy="0 0 0" />
+	</xacro:property>
+<xacro:property name="rear_right_origin">
+ 	 <origin xyz="${-wheelbase/2} ${-track/2} ${wheel_vertical_offset}" rpy="0 0 0" />
+	</xacro:property>
+    <xacro:husky_wheel wheel_prefix="front_left">
+	<origin xyz="${wheelbase/2} ${track/2} ${wheel_vertical_offset}" rpy="0 0 0" />
+	</xacro:husky_wheel>
+    <xacro:husky_wheel wheel_prefix="front_right">
+<origin xyz="${wheelbase/2} ${-track/2} ${wheel_vertical_offset}" rpy="0 0 0" />
+</xacro:husky_wheel>
+    <xacro:husky_wheel wheel_prefix="rear_left" >
+ <origin xyz="${-wheelbase/2} ${track/2} ${wheel_vertical_offset}" rpy="0 0 0" />
+</xacro:husky_wheel>
+    <xacro:husky_wheel wheel_prefix="rear_right">
+<origin xyz="${-wheelbase/2} ${-track/2} ${wheel_vertical_offset}" rpy="0 0 0" />
+</xacro:husky_wheel>
+   <xacro:husky_wheel wheel_prefix="center_left" >
+ <origin xyz="0 ${track/2} ${wheel_vertical_offset}" rpy="0 0 0" />
+</xacro:husky_wheel>
+    <xacro:husky_wheel wheel_prefix="center_right">
+<origin xyz="0 ${-track/2} ${wheel_vertical_offset}" rpy="0 0 0" />
+</xacro:husky_wheel>
     <!-- Decorations MAcro -->
-    <xacro:rover_decorate />
+    <xacro:husky_decorate />
       <xacro:property name="reflect" value="-1" />
       <!-- Spawn arm -->
@@ -96,4 +110,3 @@
         <origin xyz="0.3058 0 0.0065" rpy="0.0 0.0 -1.57" />
       </joint>
-  </xacro:macro>
 </robot>

Commit message: Bohot Ho gaya Husky AB

File: msi_2k16_17_urdf/urdf/msi.xacro (robot description, xacro)
@@ -2,6 +2,6 @@
 <robot name="mars_rover_iitb" xmlns:xacro="http://ros.org/wiki/xacro">
   <!-- Included URDF/XACRO Files -->
-  <!-- <xacro:include filename="$(find msi_2k16_17_urdf)/urdf/decorations.urdf.xacro" /> -->
-  <xacro:include filename="$(find msi_2k16_17_urdf)/urdf/wheel.urdf.xacro" />
+  <!-- <xacro:include filename="$(find husky_description)/urdf/decorations.urdf.xacro" /> -->
+  <xacro:include filename="$(find husky_description)/urdf/wheel.urdf.xacro" />
   <!--<xacro:include filename="$(find ur_description)/urdf/ur5.urdf.xacro" />-->
   <property name="M_PI" value="3.14159"/>
@@ -13,7 +13,9 @@
   <property name="wheel_L" value="0.11" />
   <property name="wheel_R" value="0.17" />
+  <property name="wheel_length" value="0.11" />
+  <property name="wheel_radius" value="0.17" />
   <!-- Wheel Mounting Positions -->
-  <xacro:property name="wheelbase" value="0.54" />
-  <xacro:property name="track" value="0.375" />
+  <xacro:property name="wheelbase" value="1.08" />
+  <xacro:property name="track" value="0.75" />
   <xacro:property name="wheel_vertical_offset" value="${-base_z_size/4}" />
     <!-- Base link is the center of the robot's bottom plate -->
@@ -28,5 +30,5 @@
     <link name="base_footprint"/>
     <joint name="base_footprint_joint" type="fixed">
-      <origin xyz="0 0 ${wheel_vertical_offset}" rpy="0 0 0" />
+      <origin xyz="0 0 ${wheel_vertical_offset - wheel_R}" rpy="0 0 0" />
       <parent link="base_link" />
       <child link="base_footprint" />
@@ -56,33 +58,36 @@
     </gazebo>
     <!-- wheel macros -->
+    <xacro:property name="front_left_origin">
+   <origin xyz="${wheelbase/2} ${track/2} ${wheel_vertical_offset}" rpy="0 0 0" />
+  </xacro:property>
 <xacro:property name="front_right_origin">
- 	 <origin xyz="${wheelbase/2} ${-track/2} ${wheel_vertical_offset}" rpy="0 0 0" />
-	</xacro:property>
+   <origin xyz="${wheelbase/2} ${-track/2} ${wheel_vertical_offset}" rpy="0 0 0" />
+  </xacro:property>
 <xacro:property name="rear_left_origin">
- 	 <origin xyz="${-wheelbase/2} ${track/2} ${wheel_vertical_offset}" rpy="0 0 0" />
-	</xacro:property>
+   <origin xyz="${-wheelbase/2} ${track/2} ${wheel_vertical_offset}" rpy="0 0 0" />
+  </xacro:property>
 <xacro:property name="rear_right_origin">
- 	 <origin xyz="${-wheelbase/2} ${-track/2} ${wheel_vertical_offset}" rpy="0 0 0" />
-	</xacro:property>
-<xacro:husky_wheel wheel_prefix="front_left">
-	<origin xyz="${wheelbase/2} ${track/2} ${wheel_vertical_offset}" rpy="0 0 0" />
-	</xacro:husky_wheel>
-<xacro:husky_wheel wheel_prefix="front_right">
-	<origin xyz="${wheelbase/2} ${-track/2} ${wheel_vertical_offset}" rpy="0 0 0" />
+   <origin xyz="${-wheelbase/2} ${-track/2} ${wheel_vertical_offset}" rpy="0 0 0" />
+  </xacro:property>
+    <xacro:husky_wheel wheel_prefix="front_left">
+  <origin xyz="${wheelbase/2} ${track/2} ${wheel_vertical_offset}" rpy="0 0 0" />
+  </xacro:husky_wheel>
+    <xacro:husky_wheel wheel_prefix="front_right">
+<origin xyz="${wheelbase/2} ${-track/2} ${wheel_vertical_offset}" rpy="0 0 0" />
 </xacro:husky_wheel>
-<xacro:husky_wheel wheel_prefix="rear_left" >
-	<origin xyz="${-wheelbase/2} ${track/2} ${wheel_vertical_offset}" rpy="0 0 0" />
+    <xacro:husky_wheel wheel_prefix="rear_left" >
+ <origin xyz="${-wheelbase/2} ${track/2} ${wheel_vertical_offset}" rpy="0 0 0" />
 </xacro:husky_wheel>
-<xacro:husky_wheel wheel_prefix="rear_right">
-	<origin xyz="${-wheelbase/2} ${-track/2} ${wheel_vertical_offset}" rpy="0 0 0" />
+    <xacro:husky_wheel wheel_prefix="rear_right">
+<origin xyz="${-wheelbase/2} ${-track/2} ${wheel_vertical_offset}" rpy="0 0 0" />
 </xacro:husky_wheel>
-<xacro:husky_wheel wheel_prefix="center_left" >
-	<origin xyz="0 ${track/2} ${wheel_vertical_offset}" rpy="0 0 0" />
+   <xacro:husky_wheel wheel_prefix="center_left" >
+ <origin xyz="0 ${track/2} ${wheel_vertical_offset}" rpy="0 0 0" />
 </xacro:husky_wheel>
-<xacro:husky_wheel wheel_prefix="center_right">
-	<origin xyz="0 ${-track/2} ${wheel_vertical_offset}" rpy="0 0 0" />
+    <xacro:husky_wheel wheel_prefix="center_right">
+<origin xyz="0 ${-track/2} ${wheel_vertical_offset}" rpy="0 0 0" />
 </xacro:husky_wheel>
     <!-- Decorations MAcro -->
-<xacro:husky_decorate />
+    <xacro:husky_decorate />
       <xacro:property name="reflect" value="-1" />
       <!-- Spawn arm -->

File: msi_2k16_17_urdf/urdf/wheel.urdf.xacro (robot description, xacro)
@@ -32,5 +32,5 @@
 				<xacro:insert_block name="joint_pose"/>
 				<geometry>
-					<mesh filename="package://msi_2k16_17_urdf/meshes/wheel.dae" />
+					<mesh filename="package://husky_description/meshes/wheel.dae" />
 				</geometry>
 			</visual>
@@ -38,5 +38,5 @@
 				<xacro:insert_block name="joint_pose"/>
 				<geometry>
-					<cylinder length="${wheel_L}" radius="${wheel_R}" />
+					<cylinder length="${wheel_length}" radius="${wheel_radius}" />
 				</geometry>
 			</collision>

Commit message: Color

File: msi_2k16_17_urdf/urdf/msi.xacro (robot description, xacro)
@@ -5,4 +5,7 @@
   <xacro:include filename="$(find husky_description)/urdf/wheel.urdf.xacro" />
   <!--<xacro:include filename="$(find ur_description)/urdf/ur5.urdf.xacro" />-->
+  <material name="chassis">
+    <color rgba="0.67 0.78 0.85 1" />
+  </material>
   <property name="M_PI" value="3.14159"/>
   <!-- Base Size -->
@@ -18,5 +21,5 @@
   <xacro:property name="wheelbase" value="1.08" />
   <xacro:property name="track" value="0.75" />
-  <xacro:property name="wheel_vertical_offset" value="${-base_z_size/4}" />
+  <xacro:property name="wheel_vertical_offset" value="${-base_z_size/2}" />
     <!-- Base link is the center of the robot's bottom plate -->
   <link name="base_link">
@@ -25,4 +28,5 @@
         <box size="${base_x_size} ${base_y_size} ${base_z_size}"/>
       </geometry>
+      <material name="chassis"/>
     </visual>
   </link>

Commit message: URDF: Alpha Version

File: msi_2k16_17_urdf/urdf/msi.xacro (robot description, xacro)
@@ -4,5 +4,5 @@
   <!-- <xacro:include filename="$(find husky_description)/urdf/decorations.urdf.xacro" /> -->
   <xacro:include filename="$(find husky_description)/urdf/wheel.urdf.xacro" />
-  <!--<xacro:include filename="$(find ur_description)/urdf/ur5.urdf.xacro" />-->
+  <xacro:include filename="$(find jaco_description)/urdf/gazebo/jaco.urdf" />
   <material name="chassis">
     <color rgba="0.67 0.78 0.85 1" />
@@ -26,5 +26,5 @@
     <visual>
       <geometry>
-        <box size="${base_x_size} ${base_y_size} ${base_z_size}"/>
+         <mesh filename="package://husky_description/meshes/base_link.dae" scale="1.5 1.5 1"/>
       </geometry>
       <material name="chassis"/>
@@ -95,12 +95,9 @@
     <xacro:husky_decorate />
       <xacro:property name="reflect" value="-1" />
-      <!-- Spawn arm -->
-<!--    <xacro:ur5_robot prefix="ur5_arm_" joint_limited="true"/> -->
       <!-- Join arm -->
-<!--      <joint name="ur5_arm_base" type="fixed">
-        <parent link="top_plate_link" />
-        <child link="ur5_arm_base_link" />
-        <origin xyz="0.3058 0 0.0065" rpy="0.0 0.0 -1.57" />
+     <joint name="jaco_arm_base" type="fixed">
+        <parent link="base_link" />
+        <child link="base_link1" />
+        <origin xyz="0.4 0 0" rpy="0 0 0" />
       </joint>
--->
 </robot>

Commit message: Final Gazebo Trial

File: msi_2k16_17_urdf/urdf/msi.xacro (robot description, xacro)
@@ -16,5 +16,5 @@
   <property name="wheel_L" value="0.18" />
   <property name="wheel_R" value="0.17" />
-  <property name="wheel_length" value="0.17" />
+  <property name="wheel_length" value="0.18" />
   <property name="wheel_radius" value="0.17" />
   <!-- Wheel Mounting Positions -->
@@ -26,6 +26,5 @@
     <visual>
       <geometry>
-         <mesh filename="package://husky_description/msi_files/chassis.stl" scale="0.01 0.01 0.01"/>
-         <!-- <mesh filename="package://msi_files/rover.stl"> -->
+         <mesh filename="package://msi_2k16_17_urdf/meshes/chassis.stl" scale="0.01 0.01 0.01"/>
       </geometry>
       <origin xyz="0 0 0" rpy="0 0 ${+M_PI/2}"/>
@@ -95,5 +94,5 @@
 </xacro:husky_wheel>
     <!-- Decorations MAcro -->
-    <xacro:husky_decorate />
+    <!-- <xacro:husky_decorate /> -->
       <xacro:property name="reflect" value="-1" />
       <!-- Join arm -->

Commit message: Rover Craxx

File: msi_2k16_17_urdf/urdf/msi.xacro (robot description, xacro)
@@ -13,4 +13,10 @@
   <property name="base_y_size" value="0.59" />
   <property name="base_z_size" value="0.35" />
+  <property name="rocker_wheel_x" value="0.4947" />
+  <property name="rocker_wheel_y" value="0.1083" />
+  <property name="rocker_wheel_z" value="-0.2738" />
+  <property name="bogie_wheel_x" value="0.2348" />
+  <property name="bogie_wheel_y" value="0.1146" />
+  <property name="bogie_wheel_z" value="-0.1932" />
   <!-- Wheel Properties -->
   <property name="wheel_L" value="0.18" />
@@ -28,9 +34,9 @@
          <mesh filename="package://msi_2k16_17_urdf/meshes/chassis.stl" scale="0.01 0.01 0.01"/>
       </geometry>
-      <origin xyz="0 0 0" rpy="0 0 ${+M_PI/2}"/>
+      <origin xyz="0 0 0" rpy="0 0 ${-M_PI/2}"/>
       <material name="chassis"/>
     </visual>
   </link>
-  <link name="rocker_left">
+  <link name="rocker_R">
      <visual>
       <geometry>
@@ -49,12 +55,12 @@
     </inertial>
   </link>
-  <joint name="rocker_left_to_chassis" type="revolute">
-      <origin xyz=" 0 ${base_y_size/2 + 0.07} 0" rpy="0 0 0"/>
+  <joint name="rocker_R_to_chassis" type="revolute">
+      <origin xyz=" 0 ${base_y_size/2 + 0.09} 0" rpy="0 0 0"/>
       <parent link="base_link"/>
-      <child link="rocker_left"/>
-<limit effort="100" lower="-0.17" upper="0.17" velocity="1"/>
+      <child link="rocker_R"/>
+<limit effort="20" lower="-0.17" upper="0.17" velocity="1"/>
       <axis xyz="0 1 0" rpy="0 0 0" />
   </joint>
-  <link name="rocker_right">
+  <link name="rocker_L">
      <visual>
       <geometry>
@@ -73,17 +79,17 @@
     </inertial>
   </link>
-  <joint name="rocker_right_to_chassis" type="revolute">
+  <joint name="rocker_L_to_chassis" type="revolute">
       <origin xyz=" 0 ${-base_y_size/2 - 0.02} 0" rpy="0 0 0"/>
       <parent link="base_link"/>
-      <child link="rocker_right"/>
-<limit effort="100" lower="-0.17" upper="0.17" velocity="1"/>
+      <child link="rocker_L"/>
+<limit effort="20" lower="-0.17" upper="0.17" velocity="1"/>
       <axis xyz="0 1 0" rpy="0 0 0" />
   </joint>
-  <link name="bogie_left">
+  <link name="bogie_R">
     <visual>
      <geometry>
        <mesh filename="package://msi_2k16_17_urdf/meshes/bogie.stl" scale="0.01 0.01 0.01"/>
      </geometry>
-      <origin xyz="-0.202 -0.0444 -0.1434" rpy="0 0 0"/>
+      <origin xyz="0 0 0" rpy="0 0 0"/>
       <material name="chassis"/>
     </visual>
@@ -97,17 +103,17 @@
     </inertial>
   </link>
-  <joint name="bogie_left_to_rocker" type="revolute">
-      <origin xyz="0 0 0 " rpy="0 0 0"/>
-      <parent link="rocker_left"/>
-      <child link="bogie_left"/>
-<limit effort="100" lower="-0.17" upper="0.17" velocity="1"/>
+  <joint name="bogie_R_to_rocker" type="revolute">
+      <origin xyz="-0.202 -0.0444 -0.1434" rpy="0 0 0"/>
+      <parent link="rocker_R"/>
+      <child link="bogie_R"/>
+<limit effort="20" lower="-0.17" upper="0.17" velocity="1"/>
       <axis xyz="0 1 0" rpy="0 0 0" />
   </joint>
-  <link name="bogie_right">
+  <link name="bogie_L">
     <visual>
      <geometry>
        <mesh filename="package://msi_2k16_17_urdf/meshes/bogie.stl" scale="0.01 0.01 0.01"/>
      </geometry>
-      <origin xyz="-0.202 -0.044 -0.1434 " rpy="0 0 0"/>
+      <origin xyz="0 0 0" rpy="0 0 0"/>
       <material name="chassis"/>
     </visual>
@@ -121,9 +127,9 @@
     </inertial>
   </link>
-  <joint name="bogie_right_to_roc" type="revolute">
-      <origin xyz="0 0 0" rpy="0 0 0"/>
-      <parent link="rocker_right"/>
-      <child link="bogie_right"/>
-<limit effort="100" lower="-0.17" upper="0.17" velocity="1"/>
+  <joint name="bogie_L_to_rocker" type="revolute">
+      <origin xyz="-0.202 -0.044 -0.1434 " rpy="0 0 0"/>
+      <parent link="rocker_L"/>
+      <child link="bogie_L"/>
+<limit effort="20" lower="-0.17" upper="0.17" velocity="1"/>
       <axis xyz="0 1 0" rpy="0 0 0" />
   </joint>
@@ -159,34 +165,22 @@
     </gazebo>
     <!-- wheel macros -->
-    <xacro:property name="front_left_origin">
-   <origin xyz="${wheelbase/2} ${track/2} ${wheel_vertical_offset}" rpy="0 0 0" />
-  </xacro:property>
-<xacro:property name="front_right_origin">
-   <origin xyz="${wheelbase/2} ${-track/2} ${wheel_vertical_offset}" rpy="0 0 0" />
-  </xacro:property>
-<xacro:property name="rear_left_origin">
-   <origin xyz="${-wheelbase/2} ${track/2} ${wheel_vertical_offset}" rpy="0 0 0" />
-  </xacro:property>
-<xacro:property name="rear_right_origin">
-   <origin xyz="${-wheelbase/2} ${-track/2} ${wheel_vertical_offset}" rpy="0 0 0" />
-  </xacro:property>
-    <xacro:husky_wheel wheel_prefix="front_left">
-  <origin xyz="${wheelbase/2} ${track/2} ${wheel_vertical_offset}" rpy="0 0 0" />
-  </xacro:husky_wheel>
-    <xacro:husky_wheel wheel_prefix="front_right">
-<origin xyz="${wheelbase/2} ${-track/2} ${wheel_vertical_offset}" rpy="0 0 0" />
-</xacro:husky_wheel>
-    <xacro:husky_wheel wheel_prefix="rear_left" >
- <origin xyz="${-wheelbase/2} ${track/2} ${wheel_vertical_offset}" rpy="0 0 0" />
-</xacro:husky_wheel>
-    <xacro:husky_wheel wheel_prefix="rear_right">
-<origin xyz="${-wheelbase/2} ${-track/2} ${wheel_vertical_offset}" rpy="0 0 0" />
-</xacro:husky_wheel>
-   <xacro:husky_wheel wheel_prefix="center_left" >
- <origin xyz="0 ${track/2} ${wheel_vertical_offset}" rpy="0 0 0" />
-</xacro:husky_wheel>
-    <xacro:husky_wheel wheel_prefix="center_right">
-<origin xyz="0 ${-track/2} ${wheel_vertical_offset}" rpy="0 0 0" />
-</xacro:husky_wheel>
+    <xacro:husky_wheel wheel_prefix="front_L" parent="bogie_L">
+  <origin xyz="${-bogie_wheel_x} ${-bogie_wheel_y} ${bogie_wheel_z}" rpy="0 0 0" />
+    </xacro:husky_wheel>
+    <xacro:husky_wheel wheel_prefix="front_R" parent="bogie_R">
+  <origin xyz="${-bogie_wheel_x} ${bogie_wheel_y} ${bogie_wheel_z}" rpy="0 0 0" />
+    </xacro:husky_wheel>
+    <xacro:husky_wheel wheel_prefix="rear_L" parent="rocker_L">
+  <origin xyz="${rocker_wheel_x} ${-rocker_wheel_y} ${rocker_wheel_z}" rpy="0 0 0" />
+    </xacro:husky_wheel>
+    <xacro:husky_wheel wheel_prefix="rear_R" parent="rocker_R">
+  <origin xyz="${rocker_wheel_x} ${rocker_wheel_y} ${rocker_wheel_z}" rpy="0 0 0" />
+    </xacro:husky_wheel>
+    <xacro:husky_wheel wheel_prefix="center_L" parent="bogie_L">
+  <origin xyz="${bogie_wheel_x} ${-bogie_wheel_y} ${bogie_wheel_z}" rpy="0 0 0" />
+    </xacro:husky_wheel>
+    <xacro:husky_wheel wheel_prefix="center_R" parent="bogie_R">
+  <origin xyz="${bogie_wheel_x} ${bogie_wheel_y} ${bogie_wheel_z}" rpy="0 0 0" />
+    </xacro:husky_wheel>
     <!-- Decorations MAcro -->
     <!-- <xacro:husky_decorate /> -->
@@ -196,5 +190,5 @@
         <parent link="base_link" />
         <child link="base_link1" />
-        <origin xyz="${base_x_size -0.7} 0 0" rpy="0 0 0" />
+        <origin xyz=" -0.2 0 0" rpy="0 0 ${M_PI}" />
       </joint>
 </robot>

File: msi_2k16_17_urdf/urdf/wheel.urdf.xacro (robot description, xacro)
@@ -22,8 +22,8 @@
 -->
 <robot xmlns:xacro="http://ros.org/wiki/xacro" name="husky_wheel">
-	<xacro:macro name="husky_wheel" params="wheel_prefix *joint_pose">
+	<xacro:macro name="husky_wheel" params="wheel_prefix *joint_pose parent">
 		<link name="${wheel_prefix}_wheel_link">
 			<inertial>
-				<mass value="2.637" />
+				<mass value="5" />
 				<origin xyz="0 0 0" />
 				<inertia  ixx="0.02467" ixy="0" ixz="0" iyy="0.02467" iyz="0" izz="0.04411" />
@@ -50,5 +50,5 @@
 		</gazebo>
 		<joint name="${wheel_prefix}_wheel" type="continuous">
-			<parent link="base_link"/>
+			<parent link="${parent}"/>
 			<child link="${wheel_prefix}_wheel_link"/>
 			<xacro:insert_block name="joint_pose"/>
