Commit message: Differential v1

File: msi_2k16_17_urdf/urdf/msi.xacro (robot description, xacro)
@@ -56,5 +56,5 @@
   </link>
   <joint name="rocker_R_to_chassis" type="revolute">
-      <origin xyz=" 0 ${base_y_size/2 + 0.09} 0" rpy="0 0 0"/>
+      <origin xyz=" 0 ${base_y_size/2 + 0.02} 0" rpy="0 0 0"/>
       <parent link="base_link"/>
       <child link="rocker_R"/>
@@ -186,4 +186,135 @@
     <!-- <xacro:husky_decorate /> -->
       <xacro:property name="reflect" value="-1" />
+      <!-- Differential Suspension -->
+      <link name="diff_rod_main" >
+         <visual>
+          <geometry>
+             <mesh filename="package://msi_2k16_17_urdf/meshes/rod.stl" scale="0.01 0.01 0.01"/>
+          </geometry>
+          <origin xyz="0 0 0" rpy="0 0 0"/>
+          <material name="chassis"/>
+        </visual>
+        <inertial>
+          <origin xyz="0 0 0" rpy="0 0 0"/>
+          <mass value="1"/>
+          <inertia
+            ixx="1.0" ixy="0.0" ixz="0.0"
+            iyy="1.0" iyz="0.0"
+            izz="1.0"/>
+        </inertial>
+      </link>
+      <link name="diff_rod_side1" >
+         <visual>
+          <geometry>
+             <mesh filename="package://msi_2k16_17_urdf/meshes/srod.stl" scale="0.01 0.01 0.01"/>
+          </geometry>
+          <origin xyz="0 0 0" rpy="0 0 0"/>
+          <material name="chassis"/>
+        </visual>
+        <inertial>
+          <origin xyz="0 0 0" rpy="0 0 0"/>
+          <mass value="1"/>
+          <inertia
+            ixx="1.0" ixy="0.0" ixz="0.0"
+            iyy="1.0" iyz="0.0"
+            izz="1.0"/>
+        </inertial>
+      </link>
+      <link name="diff_rod_side2" >
+         <visual>
+          <geometry>
+             <mesh filename="package://msi_2k16_17_urdf/meshes/srod.stl" scale="0.01 0.01 0.01"/>
+          </geometry>
+          <origin xyz="0 0 0" rpy="0 0 0"/>
+          <material name="chassis"/>
+        </visual>
+        <inertial>
+          <origin xyz="0 0 0" rpy="0 0 0"/>
+          <mass value="1"/>
+          <inertia
+            ixx="1.0" ixy="0.0" ixz="0.0"
+            iyy="1.0" iyz="0.0"
+            izz="1.0"/>
+        </inertial>
+      </link>
+      <link name="triangle" >
+         <visual>
+          <geometry>
+             <mesh filename="package://msi_2k16_17_urdf/meshes/triangle.stl" scale="0.01 0.01 0.01"/>
+          </geometry>
+          <origin xyz="0 0 0" rpy="0 0 0"/>
+          <material name="chassis"/>
+        </visual>
+        <inertial>
+          <origin xyz="0 0 0" rpy="0 0 0 "/>
+          <mass value="1"/>
+          <inertia
+            ixx="1.0" ixy="0.0" ixz="0.0"
+            iyy="1.0" iyz="0.0"
+            izz="1.0"/>
+        </inertial>
+      </link>
+      <link name="triangle_MIR" >
+         <visual>
+          <geometry>
+             <mesh filename="package://msi_2k16_17_urdf/meshes/triangle_MIR.stl" scale="0.01 0.01 0.01"/>
+          </geometry>
+        <origin xyz="0 0 0" rpy="0 0 0"/>
+          <material name="chassis"/>
+        </visual>
+        <inertial>
+          <origin xyz="0 0 0" rpy="0 0 0"/>
+          <mass value="1"/>
+          <inertia
+            ixx="1.0" ixy="0.0" ixz="0.0"
+            iyy="1.0" iyz="0.0"
+            izz="1.0"/>
+        </inertial>
+      </link>
+      <!-- joints for differential -->
+      <joint name="triangle_to_chassis" type="fixed">
+                  <origin xyz="${(base_x_size/2-0.0143)} 0.2023 0.0345" rpy="0 0 0"/>
+                  <parent link="base_link"/>
+                    <child link="triangle"/>
+                  </joint>
+      <joint name="triangle_MIR_to_chassis" type="fixed">
+                      <origin xyz="${(base_x_size/2-0.0143)} -0.2023 0.0345" rpy="0 0 0"/>
+                      <parent link="base_link"/>
+                        <child link="triangle_MIR"/>
+                  </joint>
+      <joint name="rod_to_triangle" type="fixed">
+            <origin xyz="-0.0143 0.2023 0.0345" rpy="0 0 0"/>
+            <parent link="diff_rod_main"/>
+            <child link="triangle"/>
+          </joint>
+      <joint name="rod_to_triangle_MIR" type="fixed">
+              <origin xyz="0.0143 0.2023 -0.0345" rpy="0 0 0"/>
+              <child link="diff_rod_main"/>
+              <parent link="triangle_MIR"/>
+            </joint>
+      <joint name="triangle_to_srod" type="revolute">
+                <origin xyz="-0.0031 0.1036 -0.0705" rpy="0 0 0"/>
+                <parent link="triangle"/>
+                <child link="diff_rod_side1"/>
+        <limit effort="20" lower="-0.10" upper="0.10" velocity="1"/>
+                <axis xyz="1 0 0" rpy="0 0 0" />
+        </joint>
+        <joint name="triangle_MIR_to_srod" type="revolute">
+                  <origin xyz="-0.0031 -0.1036 -0.0705" rpy="0 0 0"/>
+                  <parent link="triangle_MIR"/>
+                  <child link="diff_rod_side2"/>
+          <limit effort="20" lower="-0.10" upper="0.10" velocity="1"/>
+                  <axis xyz="1 0 0" rpy="0 0 0" />
+          </joint>
+        <joint name="srod1_to_rockerR" type="fixed">
+                      <origin xyz="${-base_x_size/2+0.0174} ${+base_y_size/2-0.3059} 0.0360" rpy="0 0 0"/>
+                      <parent link="diff_rod_side1"/>
+                      <child link="rocker_R"/>
+        </joint>
+        <joint name="srod2_to_rockerL" type="fixed">
+                      <origin xyz="${-base_x_size/2+0.0174} ${-base_y_size/2+0.3059} 0.0360" rpy="0 0 0"/>
+                      <parent link="diff_rod_side2"/>
+                      <child link="rocker_L"/>
+        </joint>
       <!-- Join arm -->
      <joint name="jaco_arm_base" type="fixed">

Commit message: Rocker MIR resolved

File: msi_2k16_17_urdf/urdf/msi.xacro (robot description, xacro)
@@ -41,5 +41,5 @@
      <visual>
       <geometry>
-         <mesh filename="package://msi_2k16_17_urdf/meshes/rocker.stl" scale="0.01 0.01 0.01"/>
+         <mesh filename="package://msi_2k16_17_urdf/meshes/rocker_MIR.stl" scale="0.01 0.01 0.01"/>
       </geometry>
       <origin xyz="0 0 0" rpy="0 0 0"/>
@@ -56,5 +56,5 @@
   </link>
   <joint name="rocker_R_to_chassis" type="revolute">
-      <origin xyz=" 0 ${base_y_size/2 + 0.02} 0" rpy="0 0 0"/>
+      <origin xyz=" 0 ${base_y_size/2 + 0.04} 0" rpy="0 0 0"/>
       <parent link="base_link"/>
       <child link="rocker_R"/>
@@ -104,5 +104,5 @@
   </link>
   <joint name="bogie_R_to_rocker" type="revolute">
-      <origin xyz="-0.202 -0.0444 -0.1434" rpy="0 0 0"/>
+      <origin xyz="-0.202 0.0200 -0.1434" rpy="0 0 0"/>
       <parent link="rocker_R"/>
       <child link="bogie_R"/>
@@ -284,15 +284,15 @@
                   </joint>
       <joint name="rod_to_triangle" type="fixed">
-            <origin xyz="-0.0143 0.2023 0.0345" rpy="0 0 0"/>
-            <parent link="diff_rod_main"/>
-            <child link="triangle"/>
+            <origin xyz="0.0114 0.2035 -0.0356" rpy="0 0 0"/>
+            <child link="diff_rod_main"/>
+            <parent link="triangle"/>
           </joint>
       <joint name="rod_to_triangle_MIR" type="fixed">
-              <origin xyz="0.0143 0.2023 -0.0345" rpy="0 0 0"/>
+              <origin xyz="0.0114 0.2035 -0.0356" rpy="0 0 0"/>
               <child link="diff_rod_main"/>
               <parent link="triangle_MIR"/>
             </joint>
       <joint name="triangle_to_srod" type="revolute">
-                <origin xyz="-0.0031 0.1036 -0.0705" rpy="0 0 0"/>
+                <origin xyz="0.0167 0.1017 -0.0729" rpy="0 0 0"/>
                 <parent link="triangle"/>
                 <child link="diff_rod_side1"/>
@@ -301,5 +301,5 @@
         </joint>
         <joint name="triangle_MIR_to_srod" type="revolute">
-                  <origin xyz="-0.0031 -0.1036 -0.0705" rpy="0 0 0"/>
+                  <origin xyz="0.0167 -0.1017 -0.0729" rpy="0 0 0"/>
                   <parent link="triangle_MIR"/>
                   <child link="diff_rod_side2"/>
@@ -308,12 +308,12 @@
           </joint>
         <joint name="srod1_to_rockerR" type="fixed">
-                      <origin xyz="${-base_x_size/2+0.0174} ${+base_y_size/2-0.3059} 0.0360" rpy="0 0 0"/>
-                      <parent link="diff_rod_side1"/>
-                      <child link="rocker_R"/>
+                      <origin xyz="${base_x_size/2-0.0281} ${-base_y_size/2+0.3052} -0.0373" rpy="0 0 0"/>
+                      <child link="diff_rod_side1"/>
+                      <parent link="rocker_R"/>
         </joint>
         <joint name="srod2_to_rockerL" type="fixed">
-                      <origin xyz="${-base_x_size/2+0.0174} ${-base_y_size/2+0.3059} 0.0360" rpy="0 0 0"/>
-                      <parent link="diff_rod_side2"/>
-                      <child link="rocker_L"/>
+                      <origin xyz="${base_x_size/2-0.0281} ${base_y_size/2-0.3052} -0.0373" rpy="0 0 0"/>
+                      <child link="diff_rod_side2"/>
+                      <parent link="rocker_L"/>
         </joint>
       <!-- Join arm -->

Commit message: Suspension on Hold

File: msi_2k16_17_urdf/urdf/msi.xacro (robot description, xacro)
@@ -273,26 +273,32 @@
       </link>
       <!-- joints for differential -->
-      <joint name="triangle_to_chassis" type="fixed">
+      <joint name="triangle_to_chassis" type="revolute">
                   <origin xyz="${(base_x_size/2-0.0143)} 0.2023 0.0345" rpy="0 0 0"/>
                   <parent link="base_link"/>
                     <child link="triangle"/>
+                    <axis xyz="1 0 0" rpy="0 0 0" />
+        <limit effort="20" lower="-0.10" upper="0.10" velocity="1"/>
                   </joint>
-      <joint name="triangle_MIR_to_chassis" type="fixed">
+      <joint name="triangle_MIR_to_chassis" type="revolute">
                       <origin xyz="${(base_x_size/2-0.0143)} -0.2023 0.0345" rpy="0 0 0"/>
                       <parent link="base_link"/>
-                        <child link="triangle_MIR"/>
+                      <child link="triangle_MIR"/>
+                      <axis xyz="1 0 0" rpy="0 0 0" />
+        <limit effort="20" lower="-0.10" upper="0.10" velocity="1"/>
                   </joint>
-      <joint name="rod_to_triangle" type="fixed">
+      <joint name="rod_to_triangle" type="continuous">
             <origin xyz="0.0114 0.2035 -0.0356" rpy="0 0 0"/>
             <child link="diff_rod_main"/>
+            <axis xyz="1 0 0" rpy="0 0 0" />
             <parent link="triangle"/>
           </joint>
-      <joint name="rod_to_triangle_MIR" type="fixed">
+      <joint name="rod_to_triangle_MIR" type="continuous">
               <origin xyz="0.0114 0.2035 -0.0356" rpy="0 0 0"/>
               <child link="diff_rod_main"/>
+              <axis xyz="1 0 0" rpy="0 0 0" />
               <parent link="triangle_MIR"/>
             </joint>
       <joint name="triangle_to_srod" type="revolute">
-                <origin xyz="0.0167 0.1017 -0.0729" rpy="0 0 0"/>
+                <origin xyz="0 0.1017 -0.0729" rpy="0 0 0"/>
                 <parent link="triangle"/>
                 <child link="diff_rod_side1"/>
@@ -307,12 +313,14 @@
                   <axis xyz="1 0 0" rpy="0 0 0" />
           </joint>
-        <joint name="srod1_to_rockerR" type="fixed">
+        <joint name="srod1_to_rockerR" type="continuous">
                       <origin xyz="${base_x_size/2-0.0281} ${-base_y_size/2+0.3052} -0.0373" rpy="0 0 0"/>
-                      <child link="diff_rod_side1"/>
+                      <child link="diff_rod_side1" />
+                      <axis xyz="1 0 0" rpy="0 0 0" />
                       <parent link="rocker_R"/>
         </joint>
-        <joint name="srod2_to_rockerL" type="fixed">
+        <joint name="srod2_to_rockerL" type="continuous">
                       <origin xyz="${base_x_size/2-0.0281} ${base_y_size/2-0.3052} -0.0373" rpy="0 0 0"/>
                       <child link="diff_rod_side2"/>
+                      <axis xyz="1 0 0" rpy="0 0 0" />
                       <parent link="rocker_L"/>
         </joint>

Commit message: Differential katta

File: msi_2k16_17_urdf/urdf/msi.xacro (robot description, xacro)
@@ -187,8 +187,8 @@
       <xacro:property name="reflect" value="-1" />
       <!-- Differential Suspension -->
-      <link name="diff_rod_main" >
+      <link name="differential" >
          <visual>
           <geometry>
-             <mesh filename="package://msi_2k16_17_urdf/meshes/rod.stl" scale="0.01 0.01 0.01"/>
+             <mesh filename="package://msi_2k16_17_urdf/meshes/differential.stl" scale="0.01 0.01 0.01"/>
           </geometry>
           <origin xyz="0 0 0" rpy="0 0 0"/>
@@ -204,117 +204,10 @@
         </inertial>
       </link>
-      <link name="diff_rod_side1" >
-         <visual>
-          <geometry>
-             <mesh filename="package://msi_2k16_17_urdf/meshes/srod.stl" scale="0.01 0.01 0.01"/>
-          </geometry>
-          <origin xyz="0 0 0" rpy="0 0 0"/>
-          <material name="chassis"/>
-        </visual>
-        <inertial>
-          <origin xyz="0 0 0" rpy="0 0 0"/>
-          <mass value="1"/>
-          <inertia
-            ixx="1.0" ixy="0.0" ixz="0.0"
-            iyy="1.0" iyz="0.0"
-            izz="1.0"/>
-        </inertial>
-      </link>
-      <link name="diff_rod_side2" >
-         <visual>
-          <geometry>
-             <mesh filename="package://msi_2k16_17_urdf/meshes/srod.stl" scale="0.01 0.01 0.01"/>
-          </geometry>
-          <origin xyz="0 0 0" rpy="0 0 0"/>
-          <material name="chassis"/>
-        </visual>
-        <inertial>
-          <origin xyz="0 0 0" rpy="0 0 0"/>
-          <mass value="1"/>
-          <inertia
-            ixx="1.0" ixy="0.0" ixz="0.0"
-            iyy="1.0" iyz="0.0"
-            izz="1.0"/>
-        </inertial>
-      </link>
-      <link name="triangle" >
-         <visual>
-          <geometry>
-             <mesh filename="package://msi_2k16_17_urdf/meshes/triangle.stl" scale="0.01 0.01 0.01"/>
-          </geometry>
-          <origin xyz="0 0 0" rpy="0 0 0"/>
-          <material name="chassis"/>
-        </visual>
-        <inertial>
-          <origin xyz="0 0 0" rpy="0 0 0 "/>
-          <mass value="1"/>
-          <inertia
-            ixx="1.0" ixy="0.0" ixz="0.0"
-            iyy="1.0" iyz="0.0"
-            izz="1.0"/>
-        </inertial>
-      </link>
-      <link name="triangle_MIR" >
-         <visual>
-          <geometry>
-             <mesh filename="package://msi_2k16_17_urdf/meshes/triangle_MIR.stl" scale="0.01 0.01 0.01"/>
-          </geometry>
-        <origin xyz="0 0 0" rpy="0 0 0"/>
-          <material name="chassis"/>
-        </visual>
-        <inertial>
-          <origin xyz="0 0 0" rpy="0 0 0"/>
-          <mass value="1"/>
-          <inertia
-            ixx="1.0" ixy="0.0" ixz="0.0"
-            iyy="1.0" iyz="0.0"
-            izz="1.0"/>
-        </inertial>
-      </link>
-      <!-- joints for differential -->
-      <joint name="triangle_to_chassis" type="fixed">
-                  <origin xyz="${(base_x_size/2-0.0143)} 0.2023 0.0345" rpy="0 0 0"/>
+      <!-- STATIC joints for differential -->
+      <joint name="diff_to_chassis" type="fixed">
+                  <origin xyz="${base_x_size/2-0.12} 0 0" rpy="0 0 0"/>
                   <parent link="base_link"/>
-                    <child link="triangle"/>
+                    <child link="differential"/>
                   </joint>
-      <joint name="triangle_MIR_to_chassis" type="fixed">
-                      <origin xyz="${(base_x_size/2-0.0143)} -0.2023 0.0345" rpy="0 0 0"/>
-                      <parent link="base_link"/>
-                        <child link="triangle_MIR"/>
-                  </joint>
-      <joint name="rod_to_triangle" type="fixed">
-            <origin xyz="0.0114 0.2035 -0.0356" rpy="0 0 0"/>
-            <child link="diff_rod_main"/>
-            <parent link="triangle"/>
-          </joint>
-      <joint name="rod_to_triangle_MIR" type="fixed">
-              <origin xyz="0.0114 0.2035 -0.0356" rpy="0 0 0"/>
-              <child link="diff_rod_main"/>
-              <parent link="triangle_MIR"/>
-            </joint>
-      <joint name="triangle_to_srod" type="revolute">
-                <origin xyz="0.0167 0.1017 -0.0729" rpy="0 0 0"/>
-                <parent link="triangle"/>
-                <child link="diff_rod_side1"/>
-        <limit effort="20" lower="-0.10" upper="0.10" velocity="1"/>
-                <axis xyz="1 0 0" rpy="0 0 0" />
-        </joint>
-        <joint name="triangle_MIR_to_srod" type="revolute">
-                  <origin xyz="0.0167 -0.1017 -0.0729" rpy="0 0 0"/>
-                  <parent link="triangle_MIR"/>
-                  <child link="diff_rod_side2"/>
-          <limit effort="20" lower="-0.10" upper="0.10" velocity="1"/>
-                  <axis xyz="1 0 0" rpy="0 0 0" />
-          </joint>
-        <joint name="srod1_to_rockerR" type="fixed">
-                      <origin xyz="${base_x_size/2-0.0281} ${-base_y_size/2+0.3052} -0.0373" rpy="0 0 0"/>
-                      <child link="diff_rod_side1"/>
-                      <parent link="rocker_R"/>
-        </joint>
-        <joint name="srod2_to_rockerL" type="fixed">
-                      <origin xyz="${base_x_size/2-0.0281} ${base_y_size/2-0.3052} -0.0373" rpy="0 0 0"/>
-                      <child link="diff_rod_side2"/>
-                      <parent link="rocker_L"/>
-        </joint>
       <!-- Join arm -->
      <joint name="jaco_arm_base" type="fixed">
