Commit message: Individual Steer Implemented in GUI

File: msi_2k16_17_urdf/urdf/msi.xacro (robot description, xacro)
@@ -117,4 +117,106 @@
      <geometry>
        <mesh filename="package://msi_2k16_17_urdf/meshes/bogie.stl" scale="0.01 0.01 0.01"/>
+     </geometry>
+      <origin xyz="0 0 0" rpy="0 0 0"/>
+      <material name="chassis"/>
+    </visual>
+    <inertial>
+      <origin xyz="0 0 1" rpy="0 0 0"/>
+      <mass value="1"/>
+      <inertia
+        ixx="1.0" ixy="0.0" ixz="0.0"
+        iyy="1.0" iyz="0.0"
+        izz="1.0"/>
+    </inertial>
+  </link>
+  <link name="steer_wheel_fL">
+    <visual>
+     <geometry>
+       <mesh filename="package://msi_2k16_17_urdf/meshes/steer_wheel_l.stl" scale="0.01 0.01 0.01"/>
+     </geometry>
+      <origin xyz="0 0 0" rpy="0 0 0"/>
+      <material name="chassis"/>
+    </visual>
+    <inertial>
+      <origin xyz="0 0 1" rpy="0 0 0"/>
+      <mass value="1"/>
+      <inertia
+        ixx="1.0" ixy="0.0" ixz="0.0"
+        iyy="1.0" iyz="0.0"
+        izz="1.0"/>
+    </inertial>
+  </link>
+  <link name="steer_wheel_fR">
+    <visual>
+     <geometry>
+       <mesh filename="package://msi_2k16_17_urdf/meshes/steer_wheel_r.stl" scale="0.01 0.01 0.01"/>
+     </geometry>
+      <origin xyz="0 0 0" rpy="0 0 0"/>
+      <material name="chassis"/>
+    </visual>
+    <inertial>
+      <origin xyz="0 0 1" rpy="0 0 0"/>
+      <mass value="1"/>
+      <inertia
+        ixx="1.0" ixy="0.0" ixz="0.0"
+        iyy="1.0" iyz="0.0"
+        izz="1.0"/>
+    </inertial>
+  </link>
+  <link name="steer_wheel_bL">
+    <visual>
+     <geometry>
+       <mesh filename="package://msi_2k16_17_urdf/meshes/steer_wheel_l.stl" scale="0.01 0.01 0.01"/>
+     </geometry>
+      <origin xyz="0 0 0" rpy="0 0 0"/>
+      <material name="chassis"/>
+    </visual>
+    <inertial>
+      <origin xyz="0 0 1" rpy="0 0 0"/>
+      <mass value="1"/>
+      <inertia
+        ixx="1.0" ixy="0.0" ixz="0.0"
+        iyy="1.0" iyz="0.0"
+        izz="1.0"/>
+    </inertial>
+  </link>
+  <link name="steer_wheel_bR">
+    <visual>
+     <geometry>
+       <mesh filename="package://msi_2k16_17_urdf/meshes/steer_wheel_r.stl" scale="0.01 0.01 0.01"/>
+     </geometry>
+      <origin xyz="0 0 0" rpy="0 0 0"/>
+      <material name="chassis"/>
+    </visual>
+    <inertial>
+      <origin xyz="0 0 1" rpy="0 0 0"/>
+      <mass value="1"/>
+      <inertia
+        ixx="1.0" ixy="0.0" ixz="0.0"
+        iyy="1.0" iyz="0.0"
+        izz="1.0"/>
+    </inertial>
+  </link>
+  <link name="drive_wheel_R">
+    <visual>
+     <geometry>
+       <mesh filename="package://msi_2k16_17_urdf/meshes/drive_wheel_l.stl" scale="0.01 0.01 0.01"/>
+     </geometry>
+      <origin xyz="0 0 0" rpy="0 0 0"/>
+      <material name="chassis"/>
+    </visual>
+    <inertial>
+      <origin xyz="0 0 1" rpy="0 0 0"/>
+      <mass value="1"/>
+      <inertia
+        ixx="1.0" ixy="0.0" ixz="0.0"
+        iyy="1.0" iyz="0.0"
+        izz="1.0"/>
+    </inertial>
+  </link>
+  <link name="drive_wheel_L">
+    <visual>
+     <geometry>
+       <mesh filename="package://msi_2k16_17_urdf/meshes/drive_wheel_r.stl" scale="0.01 0.01 0.01"/>
      </geometry>
       <origin xyz="0 0 0" rpy="0 0 0"/>
@@ -168,22 +270,133 @@
     </gazebo>
     <!-- wheel macros -->
-    <xacro:husky_wheel wheel_prefix="front_L" parent="bogie_L">
-  <origin xyz="${-bogie_wheel_x} ${-bogie_wheel_y} ${bogie_wheel_z}" rpy="0 0 0" />
+     <!-- STATIC joints for steer assembly -->
+      <joint name="bogie_to_steer_L" type="fixed">
+  			<origin xyz="${-bogie_wheel_x} 0 ${bogie_wheel_z+0.2}" rpy="0 0 0" />
+            <parent link="bogie_L"/>
+            <child link="steer_wheel_fL"/>
+        </joint>
+      <joint name="bogie_to_steer_R" type="fixed">
+        <origin xyz="${-bogie_wheel_x} 0 ${bogie_wheel_z+0.2}" rpy="0 0 0" />
+            <parent link="bogie_R"/>
+            <child link="steer_wheel_fR"/>
+        </joint>
+        <joint name="rocker_to_steer_R" type="fixed">
+              <origin xyz="${rocker_wheel_x} 0 ${rocker_wheel_z+0.2}" rpy="0 0 0" />
+              <parent link="rocker_R"/>
+              <child link="steer_wheel_bR"/>
+        </joint>
+        <joint name="rocker_to_steer_L" type="fixed">
+            <origin xyz="${rocker_wheel_x} 0 ${rocker_wheel_z+0.2}" rpy="0 0 0" />
+            <parent link="rocker_L"/>
+            <child link="steer_wheel_bL"/>
+      </joint>
+   <joint name="bogie_to_drive_L" type="fixed">
+        <origin xyz="${bogie_wheel_x} 0.1 ${bogie_wheel_z+0.05}" rpy="0 0 0" />
+            <parent link="bogie_L"/>
+            <child link="drive_wheel_L"/>
+        </joint>
+      <joint name="bogie_to_drive_R" type="fixed">
+        <origin xyz="${bogie_wheel_x} -0.1 ${bogie_wheel_z+0.05}" rpy="0 0 0" />
+            <parent link="bogie_R"/>
+            <child link="drive_wheel_R"/>
+        </joint>
+      <!-- Join arm -->
+    <xacro:husky_wheel wheel_prefix="front_L" parent="steer_wheel_fL">
+  <origin xyz="0.04 -0.13 -0.22" rpy="0 0 0" />
     </xacro:husky_wheel>
-    <xacro:husky_wheel wheel_prefix="front_R" parent="bogie_R">
-  <origin xyz="${-bogie_wheel_x} ${bogie_wheel_y} ${bogie_wheel_z}" rpy="0 0 0" />
+   <xacro:husky_wheel wheel_prefix="front_R" parent="steer_wheel_fR">
+  <origin xyz="-0.04 0.13 -0.22" rpy="0 0 0" />
     </xacro:husky_wheel>
-    <xacro:husky_wheel wheel_prefix="rear_L" parent="rocker_L">
-  <origin xyz="${rocker_wheel_x} ${-rocker_wheel_y} ${rocker_wheel_z}" rpy="0 0 0" />
+   <xacro:husky_wheel wheel_prefix="rear_L" parent="steer_wheel_bL">
+  <origin xyz="0.04 -0.13 -0.22" rpy="0 0 0" />
     </xacro:husky_wheel>
-    <xacro:husky_wheel wheel_prefix="rear_R" parent="rocker_R">
-  <origin xyz="${rocker_wheel_x} ${rocker_wheel_y} ${rocker_wheel_z}" rpy="0 0 0" />
+   <xacro:husky_wheel wheel_prefix="rear_R" parent="steer_wheel_bR">
+  <origin xyz="-0.04 0.13 -0.22" rpy="0 0 0" />
     </xacro:husky_wheel>
-    <xacro:husky_wheel wheel_prefix="center_L" parent="bogie_L">
-  <origin xyz="${bogie_wheel_x} ${-bogie_wheel_y} ${bogie_wheel_z}" rpy="0 0 0" />
-    </xacro:husky_wheel>
-    <xacro:husky_wheel wheel_prefix="center_R" parent="bogie_R">
-  <origin xyz="${bogie_wheel_x} ${bogie_wheel_y} ${bogie_wheel_z}" rpy="0 0 0" />
-    </xacro:husky_wheel>
+  <!-- Center Wheel Handled Separately; Only Drive, no Steer -->
+   <link name="center_wheel_link_L">
+      <inertial>
+        <mass value="5" />
+        <origin xyz="0 0 0" />
+        <inertia  ixx="0.02467" ixy="0" ixz="0" iyy="0.02467" iyz="0" izz="0.04411" />
+      </inertial>
+      <visual>
+        <origin xyz="0 ${-wheel_L/2} 0" rpy="0 0 ${M_PI/2}" />
+        <geometry>
+          <mesh filename="package://msi_2k16_17_urdf/meshes/tyre.stl" scale="0.01 0.01 0.01" />
+        </geometry>
+      </visual>
+      <collision>
+        <origin xyz="0 0 0" rpy="${M_PI/2} 0 0" />
+        <geometry>
+          <cylinder length="${wheel_length}" radius="${wheel_radius}" />
+        </geometry>
+      </collision>
+    </link>
+    <link name="center_wheel_link_R">
+      <inertial>
+        <mass value="5" />
+        <origin xyz="0 0 0" />
+        <inertia  ixx="0.02467" ixy="0" ixz="0" iyy="0.02467" iyz="0" izz="0.04411" />
+      </inertial>
+      <visual>
+        <origin xyz="0 ${-wheel_L/2} 0" rpy="0 0 ${M_PI/2}" />
+        <geometry>
+          <mesh filename="package://msi_2k16_17_urdf/meshes/tyre.stl" scale="0.01 0.01 0.01" />
+        </geometry>
+      </visual>
+      <collision>
+        <origin xyz="0 0 0" rpy="${M_PI/2} 0 0" />
+        <geometry>
+          <cylinder length="${wheel_length}" radius="${wheel_radius}" />
+        </geometry>
+      </collision>
+    </link>
+    <gazebo reference="center_wheel_link_R">
+      <mu1 value="1.0"/>
+      <mu2 value="1.0"/>
+      <kp value="10000000.0" />
+      <kd value="1.0" />
+      <fdir1 value="1 0 0"/>
+        <material> Gazebo/FlatBlack</material>
+    </gazebo>
+    <gazebo reference="center_wheel_link_L">
+      <mu1 value="1.0"/>
+      <mu2 value="1.0"/>
+      <kp value="10000000.0" />
+      <kd value="1.0" />
+      <fdir1 value="1 0 0"/>
+        <material> Gazebo/FlatBlack</material>
+    </gazebo>
+    <joint name="center_wheel_drive_L" type="continuous">
+      <parent link="drive_wheel_L"/>
+      <child link="center_wheel_link_L"/>
+      <origin xyz="0 -0.23 0" rpy="0 0 0" />
+      <axis xyz="0 1 0" rpy="0 0 0" />
+    </joint>
+    <transmission name="center_wheel_L_trans" type="SimpleTransmission">
+      <type>transmission_interface/SimpleTransmission</type>
+      <actuator name="center_wheel_motor_L">
+        <mechanicalReduction>1</mechanicalReduction>
+      </actuator>
+      <joint name="center_wheel_drive_L">
+        <hardwareInterface>VelocityJointInterface</hardwareInterface>
+      </joint>
+    </transmission>
+    <joint name="center_wheel_drive_R" type="continuous">
+      <parent link="drive_wheel_R"/>
+      <child link="center_wheel_link_R"/>
+      <origin xyz="0 0.23 0" rpy="0 0 0" />
+      <axis xyz="0 1 0" rpy="0 0 0" />
+    </joint>
+    <transmission name="center_wheel_R_trans" type="SimpleTransmission">
+      <type>transmission_interface/SimpleTransmission</type>
+      <actuator name="center_wheel_motor_R">
+        <mechanicalReduction>1</mechanicalReduction>
+      </actuator>
+      <joint name="center_wheel_drive_R">
+        <hardwareInterface>VelocityJointInterface</hardwareInterface>
+      </joint>
+    </transmission>
     <!-- Decorations MAcro -->
     <!-- <xacro:husky_decorate /> -->

File: msi_2k16_17_urdf/urdf/wheel.urdf.xacro (robot description, xacro)
@@ -50,5 +50,12 @@
     		<material> Gazebo/FlatBlack</material>
 		</gazebo>
-		<joint name="${wheel_prefix}_wheel" type="continuous">
+		<joint name="${wheel_prefix}_steer" type="revolute">
+			<parent link="${parent}"/>
+			<child link="${wheel_prefix}_wheel_link"/>
+			<xacro:insert_block name="joint_pose"/>
+			<axis xyz="0 0 1" rpy="0 0 0" />
+			<limit effort="20" lower="-0.52" upper="0.52" velocity="1"/>
+		</joint>
+		<joint name="${wheel_prefix}_drive" type="continuous">
 			<parent link="${parent}"/>
 			<child link="${wheel_prefix}_wheel_link"/>

Commit message: URDF Fixed

File: msi_2k16_17_urdf/urdf/msi.xacro (robot description, xacro)
@@ -1,8 +1,14 @@
 <?xml version="1.0"?>
 <robot name="mars_rover_iitb" xmlns:xacro="http://ros.org/wiki/xacro">
+  <gazebo>
+    <plugin name="drive_controller" filename="librover_gazebo.so">
+      <topicName>"cmd_vel"</topicName>
+    </plugin>
+  </gazebo>
   <!-- Included URDF/XACRO Files -->
   <!-- <xacro:include filename="$(find husky_description)/urdf/decorations.urdf.xacro" /> -->
   <xacro:include filename="$(find msi_2k16_17_urdf)/urdf/wheel.urdf.xacro" />
-  <xacro:include filename="$(find msi_2k16_17_urdf)/urdf/arm.urdf" />
+  <!-- <xacro:include filename="$(find msi_2k16_17_urdf)/urdf/hokuyo.urdf.xacro" /> -->
+  <!--<xacro:include filename="$(find msi_2k16_17_urdf)/urdf/arm.urdf" />-->
   <material name="chassis">
     <color rgba="0.67 0.78 0.85 1" />
@@ -130,106 +136,4 @@
     </inertial>
   </link>
-  <link name="steer_wheel_fL">
-    <visual>
-     <geometry>
-       <mesh filename="package://msi_2k16_17_urdf/meshes/steer_wheel_l.stl" scale="0.01 0.01 0.01"/>
-     </geometry>
-      <origin xyz="0 0 0" rpy="0 0 0"/>
-      <material name="chassis"/>
-    </visual>
-    <inertial>
-      <origin xyz="0 0 1" rpy="0 0 0"/>
-      <mass value="1"/>
-      <inertia
-        ixx="1.0" ixy="0.0" ixz="0.0"
-        iyy="1.0" iyz="0.0"
-        izz="1.0"/>
-    </inertial>
-  </link>
-  <link name="steer_wheel_fR">
-    <visual>
-     <geometry>
-       <mesh filename="package://msi_2k16_17_urdf/meshes/steer_wheel_r.stl" scale="0.01 0.01 0.01"/>
-     </geometry>
-      <origin xyz="0 0 0" rpy="0 0 0"/>
-      <material name="chassis"/>
-    </visual>
-    <inertial>
-      <origin xyz="0 0 1" rpy="0 0 0"/>
-      <mass value="1"/>
-      <inertia
-        ixx="1.0" ixy="0.0" ixz="0.0"
-        iyy="1.0" iyz="0.0"
-        izz="1.0"/>
-    </inertial>
-  </link>
-  <link name="steer_wheel_bL">
-    <visual>
-     <geometry>
-       <mesh filename="package://msi_2k16_17_urdf/meshes/steer_wheel_l.stl" scale="0.01 0.01 0.01"/>
-     </geometry>
-      <origin xyz="0 0 0" rpy="0 0 0"/>
-      <material name="chassis"/>
-    </visual>
-    <inertial>
-      <origin xyz="0 0 1" rpy="0 0 0"/>
-      <mass value="1"/>
-      <inertia
-        ixx="1.0" ixy="0.0" ixz="0.0"
-        iyy="1.0" iyz="0.0"
-        izz="1.0"/>
-    </inertial>
-  </link>
-  <link name="steer_wheel_bR">
-    <visual>
-     <geometry>
-       <mesh filename="package://msi_2k16_17_urdf/meshes/steer_wheel_r.stl" scale="0.01 0.01 0.01"/>
-     </geometry>
-      <origin xyz="0 0 0" rpy="0 0 0"/>
-      <material name="chassis"/>
-    </visual>
-    <inertial>
-      <origin xyz="0 0 1" rpy="0 0 0"/>
-      <mass value="1"/>
-      <inertia
-        ixx="1.0" ixy="0.0" ixz="0.0"
-        iyy="1.0" iyz="0.0"
-        izz="1.0"/>
-    </inertial>
-  </link>
-  <link name="drive_wheel_R">
-    <visual>
-     <geometry>
-       <mesh filename="package://msi_2k16_17_urdf/meshes/drive_wheel_l.stl" scale="0.01 0.01 0.01"/>
-     </geometry>
-      <origin xyz="0 0 0" rpy="0 0 0"/>
-      <material name="chassis"/>
-    </visual>
-    <inertial>
-      <origin xyz="0 0 1" rpy="0 0 0"/>
-      <mass value="1"/>
-      <inertia
-        ixx="1.0" ixy="0.0" ixz="0.0"
-        iyy="1.0" iyz="0.0"
-        izz="1.0"/>
-    </inertial>
-  </link>
-  <link name="drive_wheel_L">
-    <visual>
-     <geometry>
-       <mesh filename="package://msi_2k16_17_urdf/meshes/drive_wheel_r.stl" scale="0.01 0.01 0.01"/>
-     </geometry>
-      <origin xyz="0 0 0" rpy="0 0 0"/>
-      <material name="chassis"/>
-    </visual>
-    <inertial>
-      <origin xyz="0 0 1" rpy="0 0 0"/>
-      <mass value="1"/>
-      <inertia
-        ixx="1.0" ixy="0.0" ixz="0.0"
-        iyy="1.0" iyz="0.0"
-        izz="1.0"/>
-    </inertial>
-  </link>
   <joint name="bogie_L_to_rocker" type="revolute">
       <origin xyz="-0.202 -0.044 -0.1434 " rpy="0 0 0"/>
@@ -270,133 +174,22 @@
     </gazebo>
     <!-- wheel macros -->
-     <!-- STATIC joints for steer assembly -->
-      <joint name="bogie_to_steer_L" type="fixed">
-  			<origin xyz="${-bogie_wheel_x} 0 ${bogie_wheel_z+0.2}" rpy="0 0 0" />
-            <parent link="bogie_L"/>
-            <child link="steer_wheel_fL"/>
-        </joint>
-      <joint name="bogie_to_steer_R" type="fixed">
-        <origin xyz="${-bogie_wheel_x} 0 ${bogie_wheel_z+0.2}" rpy="0 0 0" />
-            <parent link="bogie_R"/>
-            <child link="steer_wheel_fR"/>
-        </joint>
-        <joint name="rocker_to_steer_R" type="fixed">
-              <origin xyz="${rocker_wheel_x} 0 ${rocker_wheel_z+0.2}" rpy="0 0 0" />
-              <parent link="rocker_R"/>
-              <child link="steer_wheel_bR"/>
-        </joint>
-        <joint name="rocker_to_steer_L" type="fixed">
-            <origin xyz="${rocker_wheel_x} 0 ${rocker_wheel_z+0.2}" rpy="0 0 0" />
-            <parent link="rocker_L"/>
-            <child link="steer_wheel_bL"/>
-      </joint>
-   <joint name="bogie_to_drive_L" type="fixed">
-        <origin xyz="${bogie_wheel_x} 0.1 ${bogie_wheel_z+0.05}" rpy="0 0 0" />
-            <parent link="bogie_L"/>
-            <child link="drive_wheel_L"/>
-        </joint>
-      <joint name="bogie_to_drive_R" type="fixed">
-        <origin xyz="${bogie_wheel_x} -0.1 ${bogie_wheel_z+0.05}" rpy="0 0 0" />
-            <parent link="bogie_R"/>
-            <child link="drive_wheel_R"/>
-        </joint>
-      <!-- Join arm -->
-    <xacro:husky_wheel wheel_prefix="front_L" parent="steer_wheel_fL">
-  <origin xyz="0.04 -0.13 -0.22" rpy="0 0 0" />
-    </xacro:husky_wheel>
-   <xacro:husky_wheel wheel_prefix="front_R" parent="steer_wheel_fR">
-  <origin xyz="-0.04 0.13 -0.22" rpy="0 0 0" />
-    </xacro:husky_wheel>
-   <xacro:husky_wheel wheel_prefix="rear_L" parent="steer_wheel_bL">
-  <origin xyz="0.04 -0.13 -0.22" rpy="0 0 0" />
-    </xacro:husky_wheel>
-   <xacro:husky_wheel wheel_prefix="rear_R" parent="steer_wheel_bR">
-  <origin xyz="-0.04 0.13 -0.22" rpy="0 0 0" />
-    </xacro:husky_wheel>
-  <!-- Center Wheel Handled Separately; Only Drive, no Steer -->
-   <link name="center_wheel_link_L">
-      <inertial>
-        <mass value="5" />
-        <origin xyz="0 0 0" />
-        <inertia  ixx="0.02467" ixy="0" ixz="0" iyy="0.02467" iyz="0" izz="0.04411" />
-      </inertial>
-      <visual>
-        <origin xyz="0 ${-wheel_L/2} 0" rpy="0 0 ${M_PI/2}" />
-        <geometry>
-          <mesh filename="package://msi_2k16_17_urdf/meshes/tyre.stl" scale="0.01 0.01 0.01" />
-        </geometry>
-      </visual>
-      <collision>
-        <origin xyz="0 0 0" rpy="${M_PI/2} 0 0" />
-        <geometry>
-          <cylinder length="${wheel_length}" radius="${wheel_radius}" />
-        </geometry>
-      </collision>
-    </link>
-    <link name="center_wheel_link_R">
-      <inertial>
-        <mass value="5" />
-        <origin xyz="0 0 0" />
-        <inertia  ixx="0.02467" ixy="0" ixz="0" iyy="0.02467" iyz="0" izz="0.04411" />
-      </inertial>
-      <visual>
-        <origin xyz="0 ${-wheel_L/2} 0" rpy="0 0 ${M_PI/2}" />
-        <geometry>
-          <mesh filename="package://msi_2k16_17_urdf/meshes/tyre.stl" scale="0.01 0.01 0.01" />
-        </geometry>
-      </visual>
-      <collision>
-        <origin xyz="0 0 0" rpy="${M_PI/2} 0 0" />
-        <geometry>
-          <cylinder length="${wheel_length}" radius="${wheel_radius}" />
-        </geometry>
-      </collision>
-    </link>
-    <gazebo reference="center_wheel_link_R">
-      <mu1 value="1.0"/>
-      <mu2 value="1.0"/>
-      <kp value="10000000.0" />
-      <kd value="1.0" />
-      <fdir1 value="1 0 0"/>
-        <material> Gazebo/FlatBlack</material>
-    </gazebo>
-    <gazebo reference="center_wheel_link_L">
-      <mu1 value="1.0"/>
-      <mu2 value="1.0"/>
-      <kp value="10000000.0" />
-      <kd value="1.0" />
-      <fdir1 value="1 0 0"/>
-        <material> Gazebo/FlatBlack</material>
-    </gazebo>
-    <joint name="center_wheel_drive_L" type="continuous">
-      <parent link="drive_wheel_L"/>
-      <child link="center_wheel_link_L"/>
-      <origin xyz="0 -0.23 0" rpy="0 0 0" />
-      <axis xyz="0 1 0" rpy="0 0 0" />
-    </joint>
-    <transmission name="center_wheel_L_trans" type="SimpleTransmission">
-      <type>transmission_interface/SimpleTransmission</type>
-      <actuator name="center_wheel_motor_L">
-        <mechanicalReduction>1</mechanicalReduction>
-      </actuator>
-      <joint name="center_wheel_drive_L">
-        <hardwareInterface>VelocityJointInterface</hardwareInterface>
-      </joint>
-    </transmission>
-    <joint name="center_wheel_drive_R" type="continuous">
-      <parent link="drive_wheel_R"/>
-      <child link="center_wheel_link_R"/>
-      <origin xyz="0 0.23 0" rpy="0 0 0" />
-      <axis xyz="0 1 0" rpy="0 0 0" />
-    </joint>
-    <transmission name="center_wheel_R_trans" type="SimpleTransmission">
-      <type>transmission_interface/SimpleTransmission</type>
-      <actuator name="center_wheel_motor_R">
-        <mechanicalReduction>1</mechanicalReduction>
-      </actuator>
-      <joint name="center_wheel_drive_R">
-        <hardwareInterface>VelocityJointInterface</hardwareInterface>
-      </joint>
-    </transmission>
+    <xacro:husky_wheel wheel_prefix="front_L" parent="bogie_L">
+  <origin xyz="${-bogie_wheel_x} ${-bogie_wheel_y} ${bogie_wheel_z}" rpy="0 0 0" />
+    </xacro:husky_wheel>
+    <xacro:husky_wheel wheel_prefix="front_R" parent="bogie_R">
+  <origin xyz="${-bogie_wheel_x} ${bogie_wheel_y} ${bogie_wheel_z}" rpy="0 0 0" />
+    </xacro:husky_wheel>
+    <xacro:husky_wheel wheel_prefix="rear_L" parent="rocker_L">
+  <origin xyz="${rocker_wheel_x} ${-rocker_wheel_y} ${rocker_wheel_z}" rpy="0 0 0" />
+    </xacro:husky_wheel>
+    <xacro:husky_wheel wheel_prefix="rear_R" parent="rocker_R">
+  <origin xyz="${rocker_wheel_x} ${rocker_wheel_y} ${rocker_wheel_z}" rpy="0 0 0" />
+    </xacro:husky_wheel>
+    <xacro:husky_wheel wheel_prefix="center_L" parent="bogie_L">
+  <origin xyz="${bogie_wheel_x} ${-bogie_wheel_y} ${bogie_wheel_z}" rpy="0 0 0" />
+    </xacro:husky_wheel>
+    <xacro:husky_wheel wheel_prefix="center_R" parent="bogie_R">
+  <origin xyz="${bogie_wheel_x} ${bogie_wheel_y} ${bogie_wheel_z}" rpy="0 0 0" />
+    </xacro:husky_wheel>
     <!-- Decorations MAcro -->
     <!-- <xacro:husky_decorate /> -->
@@ -427,8 +220,14 @@
                   </joint>
       <!-- Join arm -->
-     <joint name="jaco_arm_base" type="fixed">
+     <!--<joint name="jaco_arm_base" type="fixed">
         <parent link="base_link" />
         <child link="base_link1" />
         <origin xyz=" -0.2 0 0" rpy="0 0 ${M_PI}" />
-      </joint>
+      </joint>-->
+<!--     <joint name="hokuyo_joint" type="fixed">
+      <origin xyz="0 0 0" rpy="0 0 0" />
+      <parent link="base_link" />
+      <child link="base_laser_link" />
+    </joint>
+ -->
 </robot>

File: msi_2k16_17_urdf/urdf/wheel.urdf.xacro (robot description, xacro)
@@ -50,12 +50,5 @@
     		<material> Gazebo/FlatBlack</material>
 		</gazebo>
-		<joint name="${wheel_prefix}_steer" type="revolute">
-			<parent link="${parent}"/>
-			<child link="${wheel_prefix}_wheel_link"/>
-			<xacro:insert_block name="joint_pose"/>
-			<axis xyz="0 0 1" rpy="0 0 0" />
-			<limit effort="20" lower="-0.52" upper="0.52" velocity="1"/>
-		</joint>
-		<joint name="${wheel_prefix}_drive" type="continuous">
+		<joint name="${wheel_prefix}_wheel" type="continuous">
 			<parent link="${parent}"/>
 			<child link="${wheel_prefix}_wheel_link"/>
