Commit message: Arm URDF feedback run

File: aspha18_urdf/urdf/aspha18.urdf (robot description, URDF)
Before this commit: robot aspha18_urdf, 9 links, 8 joints
Joints:
- joint elbow_joint: limit lower=-0.20 upper=0.20 effort=0 velocity=0 -> lower=-3.14 upper=3.14 effort=0 velocity=0
- joint gripper_joint: limit lower=-0.17 upper=0.17 effort=0 velocity=0 -> lower=-1.2 upper=1.9 effort=0 velocity=0
- joint shoulder_joint: limit lower=-0.17 upper=0.17 effort=0 velocity=0 -> lower=-0.45 upper=1.12 effort=0 velocity=0

Commit message: Kinect URDF \m/

File: aspha18_urdf/urdf/aspha18.urdf (robot description, URDF)
Before this commit: robot aspha18_urdf, 9 links, 8 joints
Links:
- added link kinect2_rgb_optical_frame, mass 2.7918; collision box size=0.1 0.6 0.1; visual box size=0.2 0.05 0.05
Joints:
- added joint kinect_joint: type fixed, parent base_link, child kinect2_rgb_optical_frame, origin xyz=0 0.35 0.12 rpy=-1.5 0 0

Commit message: wheelhub_pain sorted

File: aspha18_urdf/urdf/aspha18.urdf (robot description, URDF)
Before this commit: robot aspha18_urdf, 10 links, 9 joints
Links:
- link base_link: geometry collision mesh filename=package://rover_description/meshes/base_link.stl; visual mesh filename=package://rover_description/meshes/base_link.stl
- link base_rotn: geometry collision mesh filename=package://rover_description/meshes/base_rotn.stl; visual mesh filename=package://rover_description/meshes/base_rotn.stl
- link elbow_link: geometry collision mesh filename=package://rover_description/meshes/elbow.stl; visual mesh filename=package://rover_description/meshes/elbow.stl
- link gripper: geometry collision mesh filename=package://rover_description/meshes/gripper.stl; visual mesh filename=package://rover_description/meshes/gripper.stl
- link shoulder_links: geometry collision mesh filename=package://rover_description/meshes/shoulder.stl; visual mesh filename=package://rover_description/meshes/shoulder.stl
- link wheel1: geometry collision mesh filename=package://rover_description/meshes/wheel1.stl; visual mesh filename=package://rover_description/meshes/wheel1.stl
- link wheel2: geometry collision mesh filename=package://rover_description/meshes/wheel2.stl; visual mesh filename=package://rover_description/meshes/wheel2.stl
- link wheel3: geometry collision mesh filename=package://rover_description/meshes/wheel3.stl; visual mesh filename=package://rover_description/meshes/wheel3.stl
- link wheel4: geometry collision mesh filename=package://rover_description/meshes/wheel4.stl; visual mesh filename=package://rover_description/meshes/wheel4.stl
Joints:
- removed joint base_rot1
- removed joint rotate1
- removed joint rotate2
- removed joint rotate3
- removed joint rotate4
- added joint base_rotation: type continuous, parent base_link, child base_rotn, origin xyz=0 0.19 0.14 rpy=0 0 0, axis 0 0 1, limit effort=0 velocity=0
- added joint wheel_rotate1: type continuous, parent base_link, child wheel1, origin xyz=0.46 0.43 -0.13 rpy=0 0 0, axis 1 0 0
- added joint wheel_rotate2: type continuous, parent base_link, child wheel2, origin xyz=-0.46 0.433 -0.1345 rpy=0 0 3.14, axis 1 0 0
- added joint wheel_rotate3: type continuous, parent base_link, child wheel3, origin xyz=0.46 -0.45 -0.13 rpy=0 0 0, axis 1 0 0
- added joint wheel_rotate4: type continuous, parent base_link, child wheel4, origin xyz=-0.46 -0.435 -0.135 rpy=0 0 3.14, axis 1 0 0

Commit message: base_rotation pain sorted

File: aspha18_urdf/urdf/aspha18.urdf (robot description, URDF)
Before this commit: robot rover_description, 10 links, 9 joints
Links:
- link base_rotn: geometry collision mesh filename=package://rover_description/meshes/base_rotation.STL scale=0.001 0.001 0.001; visual mesh filename=package://rover_description/meshes/base_rotation.STL scale=0.001 0.001 0.001
Joints:
- joint base_rotation: origin xyz=0 0.19 0.14 rpy=0 0 0 -> xyz=0 0.19 0.12 rpy=0 0 0
- joint elbow_joint: origin xyz=0 0.45 0.33 rpy=-0.67 0 0 -> xyz=0 0.43 0.345 rpy=-0.67 0 0
- joint shoulder_joint: origin xyz=0 0 0.02 rpy=0 0 0 -> xyz=0 0.009 0.04 rpy=0 0 0

Commit message: bio_assembly, camera_mount, com_mount
Inertial properties update remains for the newly added components

File: aspha18_urdf/urdf/aspha18.urdf (robot description, URDF)
Before this commit: robot rover_description, 10 links, 9 joints
Links:
- added link bio_assembly, mass 5; collision mesh filename=package://rover_description/meshes/bio_assembly.STL scale=0.001 0.001 0.001; visual mesh filename=package://rover_description/meshes/bio_assembly.STL scale=0.001 0.001 0.001
- added link camera_mount, mass 5; collision mesh filename=package://rover_description/meshes/camera_mount.STL scale=0.001 0.001 0.001; visual mesh filename=package://rover_description/meshes/camera_mount.STL scale=0.001 0.001 0.001
- added link com_mount, mass 5; collision mesh filename=package://rover_description/meshes/com_mount.STL scale=0.001 0.001 0.001; visual mesh filename=package://rover_description/meshes/com_mount.STL scale=0.001 0.001 0.001
Joints:
- added joint bio_assembly_joint: type fixed, parent base_link, child bio_assembly, origin xyz=0 -0.3 0.1 rpy=0 0 0
- added joint camera_mount_joint: type fixed, parent base_link, child camera_mount, origin xyz=-0.2 0.09 0.12 rpy=0 0 0
- added joint com_mount_joint: type fixed, parent base_link, child com_mount, origin xyz=-0.15 -0.255 0.175 rpy=0 0 0

Commit message: urdf changes
added other remaining components to the urdf and posible urdf worrlds

File: aspha18_urdf/urdf/aspha18.urdf (robot description, URDF)
Before this commit: robot rover_description, 13 links, 12 joints
Links:
- link base_link: geometry collision mesh filename=package://aspha18_urdf/meshes/base_link.stl; visual mesh filename=package://aspha18_urdf/meshes/base_link.stl
- link base_rotn: geometry collision mesh filename=package://aspha18_urdf/meshes/base_rotation.STL scale=0.001 0.001 0.001; visual mesh filename=package://aspha18_urdf/meshes/base_rotation.STL scale=0.001 0.001 0.001
- link bio_assembly: geometry collision mesh filename=package://aspha18_urdf/meshes/bio_assembly.STL scale=0.001 0.001 0.001; visual mesh filename=package://aspha18_urdf/meshes/bio_assembly.STL scale=0.001 0.001 0.001
- link camera_mount: geometry collision mesh filename=package://aspha18_urdf/meshes/camera_mount.STL scale=0.001 0.001 0.001; visual mesh filename=package://aspha18_urdf/meshes/camera_mount.STL scale=0.001 0.001 0.001
- link com_mount: geometry collision mesh filename=package://aspha18_urdf/meshes/com_mount.STL scale=0.001 0.001 0.001; visual mesh filename=package://aspha18_urdf/meshes/com_mount.STL scale=0.001 0.001 0.001
- link elbow_link: geometry collision mesh filename=package://aspha18_urdf/meshes/elbow.stl; visual mesh filename=package://aspha18_urdf/meshes/elbow.stl
- link gripper: geometry collision mesh filename=package://aspha18_urdf/meshes/gripper.stl; visual mesh filename=package://aspha18_urdf/meshes/gripper.stl
- link shoulder_links: geometry collision mesh filename=package://aspha18_urdf/meshes/shoulder.stl; visual mesh filename=package://aspha18_urdf/meshes/shoulder.stl
- link wheel1: geometry collision mesh filename=package://aspha18_urdf/meshes/wheel1.stl; visual mesh filename=package://aspha18_urdf/meshes/wheel1.stl
- link wheel2: geometry collision mesh filename=package://aspha18_urdf/meshes/wheel2.stl; visual mesh filename=package://aspha18_urdf/meshes/wheel2.stl
- link wheel3: geometry collision mesh filename=package://aspha18_urdf/meshes/wheel3.stl; visual mesh filename=package://aspha18_urdf/meshes/wheel3.stl
- link wheel4: geometry collision mesh filename=package://aspha18_urdf/meshes/wheel4.stl; visual mesh filename=package://aspha18_urdf/meshes/wheel4.stl

Commit message: Adding dummy realsense fig in URDF

File: aspha18_urdf/urdf/aspha18.urdf (robot description, URDF)
Before this commit: robot aspha18_urdf, 13 links, 12 joints
Links:
- removed link kinect2_rgb_optical_frame
- added link camera_depth_frame, mass 2.7918; visual box size=0.02 0.05 0.05
Joints:
- removed joint kinect_joint
- added joint depthcam_joint: type fixed, parent gripper, child camera_depth_frame, origin xyz=0.05 0.02 -0.2 rpy=-1.5 0 0

Commit message: Adding changes to urdf for intel d435, URDF theta phi pubs

File: aspha18_urdf/urdf/aspha18.urdf (robot description, URDF)
Before this commit: robot aspha18_urdf, 13 links, 12 joints
Links:
- added link camera_color_optical_frame
- added link camera_depth_optical_frame
- added link camera_rgb_frame
- added link camera_rgb_optical_frame
- added link depthcamera_mount, mass 2.7918; visual box size=0.02 0.05 0.05
- link camera_depth_frame: mass 2.7918 -> None; geometry 
Joints:
- added joint camera_color_optical_joint: type fixed, parent camera_depth_frame, child camera_color_optical_frame, origin xyz=0 0 0 rpy=0 0 0
- added joint camera_depth_joint: type fixed, parent camera_rgb_frame, child camera_depth_frame, origin xyz=0 0 0 rpy=0 0 0
- added joint camera_depth_optical_joint: type fixed, parent camera_depth_frame, child camera_depth_optical_frame, origin xyz=0 0 0 rpy=0 0 0
- added joint camera_rgb_joint: type fixed, parent depthcamera_mount, child camera_rgb_frame, origin xyz=0 0 0 rpy=0 0 0
- added joint camera_rgb_optical_joint: type fixed, parent camera_rgb_frame, child camera_rgb_optical_frame, origin xyz=0 0 0 rpy=0 0 0
- joint depthcam_joint: child camera_depth_frame -> depthcamera_mount; origin xyz=0.05 0.02 -0.2 rpy=-1.5 0 0 -> xyz=0.05 0.02 -0.2 rpy=3.14 0 0
