Commit message: Adding Rover 19 urdf with motion feedback

File: rover19_urdf/urdf/rover19.urdf (robot description, URDF)
Before this commit: robot rover19_urdf, 9 links, 8 joints
Links:
- link base_link: geometry collision mesh filename=package://rover19_urdf/meshes/rover.stl; visual mesh filename=package://rover19_urdf/meshes/rover.stl scale=0.001 0.001 0.001
- link base_rot: geometry collision mesh filename=package://rover19_urdf/meshes/base_rot.stl; visual mesh filename=package://rover19_urdf/meshes/base_rot.stl scale=0.001 0.001 0.001
- link elbow: geometry collision mesh filename=package://rover19_urdf/meshes/elbow.stl; visual mesh filename=package://rover19_urdf/meshes/elbow.stl scale=0.001 0.001 0.001
- link finger0: geometry collision mesh filename=package://rover19_urdf/meshes/finger0.stl; visual mesh filename=package://rover19_urdf/meshes/finger0.stl scale=0.001 0.001 0.001
- link finger1: geometry collision mesh filename=package://rover19_urdf/meshes/finger1.stl; visual mesh filename=package://rover19_urdf/meshes/finger1.stl scale=0.001 0.001 0.001
- link finger2: geometry collision mesh filename=package://rover19_urdf/meshes/finger2.stl; visual mesh filename=package://rover19_urdf/meshes/finger2.stl scale=0.001 0.001 0.001
- link gripper_link1: geometry collision mesh filename=package://rover19_urdf/meshes/gripper_link1.stl; visual mesh filename=package://rover19_urdf/meshes/gripper_link1.stl scale=0.001 0.001 0.001
- link gripper_link2: geometry collision mesh filename=package://rover19_urdf/meshes/gripper_link2.stl; visual mesh filename=package://rover19_urdf/meshes/gripper_link2.stl scale=0.001 0.001 0.001
- link shoulder: geometry collision mesh filename=package://rover19_urdf/meshes/shoulder.stl; visual mesh filename=package://rover19_urdf/meshes/shoulder.stl scale=0.001 0.001 0.001
Joints:
- joint base_rot_joint: origin xyz=252.89 -15.47 246.60 rpy=0 0 0 -> xyz=0.25289 -0.01547 0.24660 rpy=0 0 0
- joint elbow_joint: origin xyz=234.16 -9.84 460.51 rpy=0 0 0 -> xyz=0.23416 -0.00984 0.46051 rpy=0 0 0
- joint finger0_joint: origin xyz=112.78 -4.82 -60.85 rpy=0 0 0 -> xyz=0.11278 -0.00482 -0.06085 rpy=0 0 0
- joint finger1_joint: origin xyz=112.78 -4.82 -60.85 rpy=0 0 0 -> xyz=0.11278 -0.00482 -0.06085 rpy=0 0 0
- joint finger2_joint: origin xyz=112.78 -4.82 -60.85 rpy=0 0 0 -> xyz=0.11278 -0.00482 -0.06085 rpy=0 0 0
- joint gripper_link1_joint: origin xyz=342.91 1.74 138.36 rpy=0 0 0 -> xyz=0.34291 0.00174 0.13836 rpy=0 0 0
- joint gripper_link2_joint: origin xyz=113.27 -4.19 -56.24 rpy=0 0 0 -> xyz=0.11327 -0.00419 -0.05624 rpy=0 0 0

Commit message: Adding depthcam mount in urdf

File: rover19_urdf/urdf/rover19.urdf (robot description, URDF)
Before this commit: robot rover19_urdf, 9 links, 8 joints
Links:
- added link camera_color_optical_frame
- added link camera_depth_frame
- added link camera_depth_optical_frame
- added link camera_rgb_frame
- added link camera_rgb_optical_frame
- added link depthcamera_mount, mass 2.7918
Joints:
- added joint camera_color_optical_joint: type fixed, parent camera_depth_frame, child camera_color_optical_frame, origin xyz=0 0 0 rpy=0 0 0
- added joint camera_depth_joint: type fixed, parent camera_rgb_frame, child camera_depth_frame, origin xyz=0 0 0 rpy=0 0 0
- added joint camera_depth_optical_joint: type fixed, parent camera_depth_frame, child camera_depth_optical_frame, origin xyz=0 0 0 rpy=0 0 0
- added joint camera_rgb_joint: type fixed, parent depthcamera_mount, child camera_rgb_frame, origin xyz=0 0 0 rpy=0 0 0
- added joint camera_rgb_optical_joint: type fixed, parent camera_rgb_frame, child camera_rgb_optical_frame, origin xyz=0 0 0 rpy=0 0 0
- added joint depthcam_joint: type fixed, parent gripper_link2, child depthcamera_mount, origin xyz=0.03252 -0.003 0.09906 rpy=0 0.7 0
